File: KiCad/_autosave-RP2040-Decoder-Rev_0_2.kicad_pcb (KiCad board)
At the start: 2 copper layers, 25 x 20 mm, 44 parts, among them J1 DCC_IN, J2 MOTOR_CONN, J3 GPIO_CONN, J4 DEBUG_CONN, Q1 WNM2030, Q2 WNM2030, Q3 WNM2030, Q4 WNM2030, U1 PJ75AL33SA, U2 BDR6133, U3 W25Q64JVSSIQ, U4 RP2040, Y1 X322512MSB4SI

Commit message: PCB & svg
Parts:
- moved C9 2.18 mm to (151.3, 104.7)
Routing:
- net /GPIO20: track 0.00 -> 15.4 mm, vias 0 -> 2
- net /GPIO21: track 0.02 -> 14.3 mm, vias 0 -> 2
Changed lines of the file:
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@@
   )
   (footprint "Capacitor_SMD:C_0603_1608Metric" (layer "F.Cu")
-    (at 149.2 104.1)
+    (at 151.3 104.7)
     (descr "Capacitor SMD 0603 (1608 Metric), square (rectangular) end terminal, IPC_7351 nominal, (Body size source: IPC-SM-782 page 76, https://www.pcb-3d.com/wordpress/wp-content/uploads/ipc-sm-782a_amendment_1_and_2.pdf), generated with kicad-footprint-generator")
     (tags "capacitor")
@@
     (property "Sheetname" "")
     (attr smd)
-    (fp_text reference "U2" (at 0 -3.4) (layer "F.SilkS")
-      (effects (font (size 1 1) (thickness 0.15)))
-    )
-    (fp_text value "BDR6133" (at 0 3.4) (layer "F.Fab")
-      (effects (font (size 1 1) (thickness 0.15)))
-    )
-    (fp_text user "${REFERENCE}" (at 0 0) (layer "F.Fab")
+    (fp_text reference "U2" (at 0 -3.4 180) (layer "F.SilkS")
+      (effects (font (size 1 1) (thickness 0.15)))
+    )
+    (fp_text value "BDR6133" (at 0 3.4 180) (layer "F.Fab")
+      (effects (font (size 1 1) (thickness 0.15)))
+    )
+    (fp_text user "${REFERENCE}" (at 0 0 180) (layer "F.Fab")
       (effects (font (size 0.98 0.98) (thickness 0.15)))
     )
+    (fp_line (start 0 2.56) (end -1.95 2.56) (layer "F.SilkS") (width 0.12))
+    (fp_line (start 0 2.56) (end 1.95 2.56) (layer "F.SilkS") (width 0.12))
     (fp_line (start 0 -2.56) (end 1.95 -2.56) (layer "F.SilkS") (width 0.12))
     (fp_line (start 0 -2.56) (end -3.45 -2.56) (layer "F.SilkS") (width 0.12))
-    (fp_line (start 0 2.56) (end -1.95 2.56) (layer "F.SilkS") (width 0.12))
-    (fp_line (start 0 2.56) (end 1.95 2.56) (layer "F.SilkS") (width 0.12))
-    (fp_line (start -3.7 -2.7) (end -3.7 2.7) (layer "F.CrtYd") (width 0.05))
     (fp_line (start 3.7 2.7) (end 3.7 -2.7) (layer "F.CrtYd") (width 0.05))
     (fp_line (start 3.7 -2.7) (end -3.7 -2.7) (layer "F.CrtYd") (width 0.05))
+    (fp_line (start -3.7 -2.7) (end -3.7 2.7) (layer "F.CrtYd") (width 0.05))
     (fp_line (start -3.7 2.7) (end 3.7 2.7) (layer "F.CrtYd") (width 0.05))
-    (fp_line (start 1.95 -2.45) (end 1.95 2.45) (layer "F.Fab") (width 0.1))
-    (fp_line (start -1.95 -1.475) (end -0.975 -2.45) (layer "F.Fab") (width 0.1))
-    (fp_line (start -0.975 -2.45) (end 1.95 -2.45) (layer "F.Fab") (width 0.1))
     (fp_line (start -1.95 2.45) (end -1.95 -1.475) (layer "F.Fab") (width 0.1))
     (fp_line (start 1.95 2.45) (end -1.95 2.45) (layer "F.Fab") (width 0.1))
+    (fp_line (start 1.95 -2.45) (end 1.95 2.45) (layer "F.Fab") (width 0.1))
+    (fp_line (start -0.975 -2.45) (end 1.95 -2.45) (layer "F.Fab") (width 0.1))
+    (fp_line (start -1.95 -1.475) (end -0.975 -2.45) (layer "F.Fab") (width 0.1))
+    (pad "" smd roundrect (at -0.6 0.825 180) (size 1.01 1.38) (layers "F.Paste") (roundrect_rratio 0.247525))
     (pad "" smd roundrect (at 0.6 0.825 180) (size 1.01 1.38) (layers "F.Paste") (roundrect_rratio 0.247525))
-    (pad "" smd roundrect (at -0.6 0.825 180) (size 1.01 1.38) (layers "F.Paste") (roundrect_rratio 0.247525))
     (pad "" smd roundrect (at 0.6 -0.825 180) (size 1.01 1.38) (layers "F.Paste") (roundrect_rratio 0.247525))
     (pad "" smd roundrect (at -0.6 -0.825 180) (size 1.01 1.38) (layers "F.Paste") (roundrect_rratio 0.247525))
@@
     (pad "8" smd roundrect (at 2.475 -1.905 180) (size 1.95 0.6) (layers "F.Cu" "F.Paste" "F.Mask") (roundrect_rratio 0.25)
       (net 21 "unconnected-(U2-Pad8)") (pinfunction "NC") (pintype "no_connect"))
-    (pad "9" thru_hole circle (at -0.7 0 180) (size 0.5 0.5) (drill 0.2) (layers *.Cu)
-      (net 4 "GND") (pinfunction "GND") (pintype "passive"))
-    (pad "9" thru_hole circle (at -0.7 1.2 180) (size 0.5 0.5) (drill 0.2) (layers *.Cu)
-      (net 4 "GND") (pinfunction "GND") (pintype "passive"))
     (pad "9" thru_hole circle (at -0.7 -1.2 180) (size 0.5 0.5) (drill 0.2) (layers *.Cu)
       (net 4 "GND") (pinfunction "GND") (pintype "passive"))
-    (pad "9" thru_hole circle (at 0.7 -1.2 180) (size 0.5 0.5) (drill 0.2) (layers *.Cu)
+    (pad "9" thru_hole circle (at 0.7 0 180) (size 0.5 0.5) (drill 0.2) (layers *.Cu)
+      (net 4 "GND") (pinfunction "GND") (pintype "passive"))
+    (pad "9" thru_hole circle (at -0.7 0 180) (size 0.5 0.5) (drill 0.2) (layers *.Cu)
       (net 4 "GND") (pinfunction "GND") (pintype "passive"))
     (pad "9" smd rect (at 0 0 180) (size 2.41 3.3) (layers "F.Cu" "F.Mask")
@@
     (pad "9" thru_hole circle (at 0.7 1.2 180) (size 0.5 0.5) (drill 0.2) (layers *.Cu)
       (net 4 "GND") (pinfunction "GND") (pintype "passive"))
+    (pad "9" thru_hole circle (at -0.7 1.2 180) (size 0.5 0.5) (drill 0.2) (layers *.Cu)
+      (net 4 "GND") (pinfunction "GND") (pintype "passive"))
+    (pad "9" thru_hole circle (at 0.7 -1.2 180) (size 0.5 0.5) (drill 0.2) (layers *.Cu)
+      (net 4 "GND") (pinfunction "GND") (pintype "passive"))
     (pad "9" smd rect (at 0 0 180) (size 1.9 2.9) (layers "B.Cu")
-      (net 4 "GND") (pinfunction "GND") (pintype "passive"))
-    (pad "9" thru_hole circle (at 0.7 0 180) (size 0.5 0.5) (drill 0.2) (layers *.Cu)
       (net 4 "GND") (pinfunction "GND") (pintype "passive"))
     (model "${KICAD6_3DMODEL_DIR}/Package_SO.3dshapes/SOIC-8-1EP_3.9x4.9mm_P1.27mm_EP2.41x3.3mm.wrl"
@@
   (segment (start 154.200498 105.87348) (end 154.936989 105.136989) (width 0.127) (layer "F.Cu") (net 37))
   (segment (start 153.177761 106.160469) (end 153.464751 105.87348) (width 0.127) (layer "F.Cu") (net 37))
+  (segment (start 159.925 108.2) (end 157.436989 108.2) (width 0.127) (layer "F.Cu") (net 38))
+  (segment (start 147.266051 105.7) (end 147.4 105.833949) (width 0.127) (layer "F.Cu") (net 38))
+  (segment (start 153.042514 105.833949) (end 153.465983 105.41048) (width 0.127) (layer "F.Cu") (net 38))
+  (segment (start 156.6 107.363011) (end 156.6 106.2) (width 0.127) (layer "F.Cu") (net 38))
+  (segment (start 147.4 105.833949) (end 153.042514 105.833949) (width 0.127) (layer "F.Cu") (net 38))
+  (segment (start 146.6375 105.7) (end 147.266051 105.7) (width 0.127) (layer "F.Cu") (net 38))
+  (segment (start 157.436989 108.2) (end 156.6 107.363011) (width 0.127) (layer "F.Cu") (net 38))
+  (segment (start 153.465983 105.41048) (end 154 105.41048) (width 0.127) (layer "F.Cu") (net 38))
+  (via (at 154 105.41048) (size 0.4) (drill 0.2) (layers "F.Cu" "B.Cu") (net 38))
+  (via (at 156.6 106.2) (size 0.4) (drill 0.2) (layers "F.Cu" "B.Cu") (net 38))
+  (segment (start 154.78952 106.2) (end 154 105.41048) (width 0.127) (layer "B.Cu") (net 38))
+  (segment (start 156.6 106.2) (end 154.78952 106.2) (width 0.127) (layer "B.Cu") (net 38))
+  (segment (start 159.925 106.1) (end 158.498989 104.673989) (width 0.127) (layer "F.Cu") (net 39))
+  (segment (start 152.907265 105.507429) (end 147.53525 105.507429) (width 0.127) (layer "F.Cu") (net 39))
   (segment (start 146.6375 105.3) (end 146.653551 105.283949) (width 0.127) (layer "F.Cu") (net 39))
+  (segment (start 153.58998 104.824713) (end 152.907265 105.507429) (width 0.127) (layer "F.Cu") (net 39))
+  (segment (start 147.327821 105.3) (end 146.6375 105.3) (width 0.127) (layer "F.Cu") (net 39))
+  (segment (start 147.53525 105.507429) (end 147.327821 105.3) (width 0.127) (layer "F.Cu") (net 39))
+  (segment (start 158.498989 104.673989) (end 157.399172 104.673989) (width 0.127) (layer "F.Cu") (net 39))
+  (segment (start 154.594483 104.824713) (end 153.58998 104.824713) (width 0.127) (layer "F.Cu") (net 39))
+  (via (at 157.399172 104.673989) (size 0.4) (drill 0.2) (layers "F.Cu" "B.Cu") (net 39))
+  (via (at 154.594483 104.824713) (size 0.4) (drill 0.2) (layers "F.Cu" "B.Cu") (net 39))
+  (segment (start 157.248448 104.824713) (end 154.594483 104.824713) (width 0.127) (layer "B.Cu") (net 39))
+  (segment (start 157.399172 104.673989) (end 157.248448 104.824713) (width 0.127) (layer "B.Cu") (net 39))
   (segment (start 139 103.982323) (end 139 104.5) (width 0.127) (layer "F.Cu") (net 53))
   (segment (start 139.282323 103.7) (end 139 103.982323) (width 0.127) (layer "F.Cu") (net 53))
