File: KiCad/RP2040-Decoder-Rev_0_2.kicad_pcb (KiCad board)
At the start: 2 copper layers, 25 x 20 mm, 57 parts, among them J1 T0, J10 2, J11 3, J12 4, J13 5, J14 +V, J15 M_OUT_B, J16 M_OUT_A, J17 GND, J18 SWCLK, J19 SWDIO, J2 T1, J20 RUN, J3 0, J4 1, J5 2, J6 3, J7 +3V3, J8 0, J9 1, Q1 T2N7002BK, Q2 T2N7002BK, Q3 T2N7002BK, Q4 T2N7002BK, Q5 T2N7002BK, U1 PJ75AL33SA, U2 BDR6133, U3 W25Q64JVSSIQ, U4 RP2040, Y1 X322512MSB4SI

Commit message: -updated docs/png -slight change to f.silkscreen
Parts:
- Q 2: renamed from Q2
- Q 3: renamed from Q3
- Q 4: renamed from Q4
- Q 5: renamed from Q5
Changed lines of the file:
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@@
     (property "Sheetname" "")
     (attr smd)
-    (fp_text reference "Q2" (at 1.3 0 90) (layer "F.SilkS")
+    (fp_text reference "Q 2" (at 1.3 0 90) (layer "F.SilkS")
       (effects (font (size 1 1) (thickness 0.15)))
     )
@@
     (property "Sheetname" "")
     (attr smd)
-    (fp_text reference "Q5" (at 1.3 0 90) (layer "F.SilkS")
+    (fp_text reference "Q 5" (at 1.3 0 90) (layer "F.SilkS")
       (effects (font (size 1 1) (thickness 0.15)))
     )
@@
     (property "Sheetname" "")
     (attr smd)
-    (fp_text reference "Q4" (at 1.3 0 90) (layer "F.SilkS")
+    (fp_text reference "Q 4" (at 1.3 0 90) (layer "F.SilkS")
       (effects (font (size 1 1) (thickness 0.15)))
     )
@@
     (property "Sheetname" "")
     (attr smd)
-    (fp_text reference "Q3" (at 1.3 0.1 90) (layer "F.SilkS")
-      (effects (font (size 1 1) (thickness 0.15)))
-    )
+    (fp_text reference "Q 3" (at 1.3 0 90) (layer "F.SilkS")
+      (effects (font (size 1 1) (thickness 0.15)))
+    )
