File: KiCad/RP2040-Decoder-Rev_0_2.kicad_sch (KiCad schematic)
At the start: 44 parts, among them J1 DCC_IN, J2 AUX_CONN, J3 GPIO_CONN, J4 DEBUG_CONN, Q1 WNM2030, Q2 WNM2030, Q3 WNM2030, Q4 WNM2030, U1 PJ75AL33SA, U2 BDR6133, U3 W25Q64JVSSIQ, U4 RP2040, Y1 X322512MSB4SI

Commit message: PCB and Schematic
Parts:
- added J3: MOTOR_CONN, Connector_PinHeader_1.00mm:PinHeader_1x04_P1.00mm_Vertical, symbol Connector:Conn_01x04_Male
- D1: Comment MBS = TO-269AA -> TO-269AA = MBS
- J1: footprint (none) -> Connector_PinHeader_1.00mm:PinHeader_1x02_P1.00mm_Vertical
- J2: footprint (none) -> Connector_PinHeader_1.00mm:PinHeader_1x04_P1.00mm_Vertical
- J4: renamed from J3; footprint (none) -> Connector_PinHeader_1.00mm:PinHeader_1x06_P1.00mm_Vertical
- J5: renamed from J4; footprint (none) -> Connector_PinHeader_1.00mm:PinHeader_1x04_P1.00mm_Vertical
- U4: footprint RP2040_minimal:RP2040-QFN-56 -> RP2040-Decoder_Additional_Footprints:QFN-56-1EP_7x7mm_P0.4mm_EP3.2x3.2mm
Connections:
- net +12V: now also U1.3 (VIN), J3.4 (Pin_4); no longer U1.2 (VI)
- net +3V3: now also C14.1, U1.2 (VOUT); no longer U1.1 (VO)
- net GND: now also J5.1 (Pin_1), Q1.2 (S), Q2.2 (S), Q3.2 (S), Q4.2 (S), U1.1 (GND), U4.19 (TESTEN), J3.1 (Pin_1); no longer J5.4 (Pin_4), U1.3 (GND)
- net at R3.2, U4.43 (ADC_AVDD): no longer C14.1
- net at J1.1 (Pin_1), R1.2: now also D1.2; no longer D1.1
- net at J1.2 (Pin_2): now also D1.1; no longer D1.2
- net MOTOR_OUT_A: now reaches R5.2, U2.4 (OUTA)
- net MOTOR_OUT_A: now also J3.3 (Pin_3)
- net MOTOR_OUT_B: now reaches R6.2, U2.5 (OUTB)
- net MOTOR_OUT_B: now also J3.2 (Pin_2)
- net at U4.26 (RUN): now also J5.2 (Pin_2); no longer J5.1 (Pin_1)
- net at U4.24 (SWCLK): now also J5.4 (Pin_4); no longer J5.2 (Pin_2)
- no-connect marks 0 -> 18
Other:
- moved on the sheet: C14

Commit message: PCB & svg
Parts:
- removed J2: AUX_CONN, Connector_PinHeader_1.00mm:PinHeader_1x04_P1.00mm_Vertical, symbol Connector:Conn_01x04_Male
- Q1, Q2, Q3, Q4: footprint Package_TO_SOT_SMD:SOT-723 -> RP2040-Decoder_Additional_Footprints:SOT-723-Extended_Pad
- renumbered J3 to J2, J4 to J3, J5 to J4
Connections:
- net +3V3: no longer C14.1
- net GPIO18: now reaches U4.29 (GPIO18)
- net GPIO18: now also Q1.1 (G)
- net GPIO19: now reaches U4.30 (GPIO19)
- net GPIO19: now also Q2.1 (G)
- net GPIO20: now reaches U4.31 (GPIO20)
- net GPIO20: now also Q3.1 (G)
- net GPIO21: now reaches U4.32 (GPIO21)
- net GPIO21: now also Q4.1 (G)
- net at R3.2, U4.43 (ADC_AVDD): now also C14.1
- net GPIO10: no longer names the net of U4.13 (GPIO10)
- net GPIO10: no longer Q1.1 (G)
- net GPIO11: no longer names the net of U4.14 (GPIO11)
- net GPIO11: no longer Q2.1 (G)
- net GPIO12: no longer names the net of U4.15 (GPIO12)
- net GPIO12: no longer Q3.1 (G)
- net GPIO13: no longer names the net of U4.16 (GPIO13)
- net GPIO13: no longer Q4.1 (G)
- no-connect marks 18 -> 22
Other:
- moved on the sheet: C14

Commit message: -changes to gitignore regarding KiCad files -changes to svg Files & Schematic ( Missing Net (GPIO) @ Input Stage)
Connections:
- net GPIO24: now reaches D2.1 (K), D3.1 (K), R2.2
- net GPIO24: now also U4.36 (GPIO24)
- no-connect marks 22 -> 21
Other:
- moved on the sheet: D2, D3, R1, R2
Changed lines of the file:
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@@
   (no_connect (at 147.32 96.52))
   (no_connect (at 147.32 149.86))
-  (no_connect (at 147.32 167.64))
   (no_connect (at 214.63 29.21))
   (no_connect (at 217.17 29.21))
@@
     (stroke (width 0) (type default) (color 0 0 0 0))
   )
-  (wire (pts (xy 137.16 167.64) (xy 147.32 167.64))
-    (stroke (width 0) (type default) (color 0 0 0 0))
-  )
   (wire (pts (xy 152.4 86.36) (xy 153.67 86.36))
     (stroke (width 0) (type default) (color 0 0 0 0))
@@
     (stroke (width 0) (type default) (color 0 0 0 0))
   )
-  (wire (pts (xy 44.45 41.91) (xy 33.02 41.91))
+  (wire (pts (xy 21.59 41.91) (xy 33.02 41.91))
     (stroke (width 0) (type default) (color 0 0 0 0))
   )
@@
     (stroke (width 0) (type default) (color 0 0 0 0))
   )
+  (wire (pts (xy 137.16 167.64) (xy 148.59 167.64))
+    (stroke (width 0) (type default) (color 0 0 0 0))
+  )
   (wire (pts (xy 106.68 86.36) (xy 106.68 88.9))
     (stroke (width 0) (type default) (color 0 0 0 0))
@@
     (stroke (width 0) (type default) (color 0 0 0 0))
   )
-  (wire (pts (xy 44.45 43.18) (xy 44.45 41.91))
+  (wire (pts (xy 21.59 43.18) (xy 21.59 41.91))
     (stroke (width 0) (type default) (color 0 0 0 0))
   )
@@
     (stroke (width 0) (type default) (color 0 0 0 0))
   )
-  (wire (pts (xy 33.02 33.02) (xy 33.02 30.48))
+  (wire (pts (xy 33.02 31.75) (xy 33.02 30.48))
     (stroke (width 0) (type default) (color 0 0 0 0))
   )
@@
     (stroke (width 0) (type default) (color 0 0 0 0))
   )
+  (wire (pts (xy 33.02 41.91) (xy 44.45 41.91))
+    (stroke (width 0) (type default) (color 0 0 0 0))
+  )
   (wire (pts (xy 67.31 78.74) (xy 67.31 77.47))
     (stroke (width 0) (type default) (color 0 0 0 0))
@@
     (stroke (width 0) (type default) (color 0 0 0 0))
   )
-  (wire (pts (xy 44.45 50.8) (xy 44.45 52.07))
+  (wire (pts (xy 21.59 50.8) (xy 21.59 52.07))
     (stroke (width 0) (type default) (color 0 0 0 0))
   )
@@
     (stroke (width 0) (type default) (color 0 0 0 0))
   )
-  (wire (pts (xy 33.02 41.91) (xy 33.02 40.64))
+  (wire (pts (xy 33.02 41.91) (xy 33.02 39.37))
     (stroke (width 0) (type default) (color 0 0 0 0))
   )
@@
     (effects (font (size 1.27 1.27)) (justify right bottom))
   )
+  (label "GPIO24" (at 44.45 41.91 180)
+    (effects (font (size 1.27 1.27)) (justify right bottom))
+  )
   (label "GPIO21" (at 245.11 39.37 0)
     (effects (font (size 1.27 1.27)) (justify left bottom))
@@
   (label "GPIO22" (at 215.9 105.41 0)
     (effects (font (size 1.27 1.27)) (justify left bottom))
+  )
+  (label "GPIO24" (at 148.59 167.64 180)
+    (effects (font (size 1.27 1.27)) (justify right bottom))
   )
   (label "GPIO18" (at 157.48 39.37 0)
@@
     (pin "2")
   )
-  (symbol (lib_id "Diode:1N4148WS") (at 33.02 36.83 270) (mirror x) (unit 1)
-    (in_bom yes) (on_board yes)
-    (property "Reference" "D2" (id 0) (at 30.988 35.6616 90)
+  (symbol (lib_id "Diode:1N4148WS") (at 33.02 35.56 90) (unit 1)
+    (in_bom yes) (on_board yes)
+    (property "Reference" "D2" (id 0) (at 35.052 34.3916 90)
       (effects (font (size 1.27 1.27)) (justify right))
     )
-    (property "Value" "1N4148WS" (id 1) (at 30.988 37.973 90)
+    (property "Value" "1N4148WS" (id 1) (at 35.052 36.703 90)
       (effects (font (size 1.27 1.27)) (justify right))
     )
-    (property "Footprint" "Diode_SMD:D_SOD-323" (id 2) (at 28.575 36.83 0)
-      (effects (font (size 1.27 1.27)) hide)
-    )
-    (property "Datasheet" "https://datasheet.lcsc.com/lcsc/2008281134_TWGMC-1N4148WS_C727111.pdf" (id 3) (at 33.02 36.83 0)
+    (property "Footprint" "Diode_SMD:D_SOD-323" (id 2) (at 37.465 35.56 0)
+      (effects (font (size 1.27 1.27)) hide)
+    )
+    (property "Datasheet" "https://datasheet.lcsc.com/lcsc/2008281134_TWGMC-1N4148WS_C727111.pdf" (id 3) (at 33.02 35.56 0)
       (effects (font (size 1.27 1.27)) hide)
     )
@@
     (pin "2")
   )
-  (symbol (lib_id "Device:R") (at 44.45 46.99 0) (mirror x) (unit 1)
-    (in_bom yes) (on_board yes)
-    (property "Reference" "R2" (id 0) (at 40.64 45.72 0))
-    (property "Value" "47k" (id 1) (at 40.64 48.26 0))
-    (property "Footprint" "Resistor_SMD:R_0603_1608Metric" (id 2) (at 42.672 46.99 90)
-      (effects (font (size 1.27 1.27)) hide)
-    )
-    (property "Datasheet" "~" (id 3) (at 44.45 46.99 0)
-      (effects (font (size 1.27 1.27)) hide)
-    )
-    (pin "1")
-    (pin "2")
-  )
-  (symbol (lib_id "Device:R") (at 33.02 26.67 0) (mirror x) (unit 1)
-    (in_bom yes) (on_board yes)
-    (property "Reference" "R1" (id 0) (at 29.21 25.4 0))
-    (property "Value" "10k" (id 1) (at 29.21 27.94 0))
-    (property "Footprint" "Resistor_SMD:R_0603_1608Metric" (id 2) (at 31.242 26.67 90)
+  (symbol (lib_id "Device:R") (at 21.59 46.99 180) (unit 1)
+    (in_bom yes) (on_board yes)
+    (property "Reference" "R2" (id 0) (at 25.4 45.72 0))
+    (property "Value" "47k" (id 1) (at 25.4 48.26 0))
+    (property "Footprint" "Resistor_SMD:R_0603_1608Metric" (id 2) (at 23.368 46.99 90)
+      (effects (font (size 1.27 1.27)) hide)
+    )
+    (property "Datasheet" "~" (id 3) (at 21.59 46.99 0)
+      (effects (font (size 1.27 1.27)) hide)
+    )
+    (pin "1")
+    (pin "2")
+  )
+  (symbol (lib_id "Device:R") (at 33.02 26.67 180) (unit 1)
+    (in_bom yes) (on_board yes)
+    (property "Reference" "R1" (id 0) (at 36.83 25.4 0))
+    (property "Value" "10k" (id 1) (at 36.83 27.94 0))
+    (property "Footprint" "Resistor_SMD:R_0603_1608Metric" (id 2) (at 34.798 26.67 90)
       (effects (font (size 1.27 1.27)) hide)
     )
@@
     (pin "2")
   )
-  (symbol (lib_id "power:GND") (at 33.02 52.07 0) (unit 1)
+  (symbol (lib_id "power:GND") (at 33.02 52.07 0) (mirror y) (unit 1)
     (in_bom yes) (on_board yes) (fields_autoplaced)
     (property "Reference" "#PWR09" (id 0) (at 33.02 58.42 0)
@@
     (pin "1")
   )
-  (symbol (lib_id "power:GND") (at 44.45 52.07 0) (unit 1)
+  (symbol (lib_id "power:GND") (at 21.59 52.07 0) (mirror y) (unit 1)
     (in_bom yes) (on_board yes) (fields_autoplaced)
-    (property "Reference" "#PWR010" (id 0) (at 44.45 58.42 0)
-      (effects (font (size 1.27 1.27)) hide)
-    )
-    (property "Value" "GND" (id 1) (at 44.45 57.15 0))
-    (property "Footprint" "" (id 2) (at 44.45 52.07 0)
-      (effects (font (size 1.27 1.27)) hide)
-    )
-    (property "Datasheet" "" (id 3) (at 44.45 52.07 0)
+    (property "Reference" "#PWR010" (id 0) (at 21.59 58.42 0)
+      (effects (font (size 1.27 1.27)) hide)
+    )
+    (property "Value" "GND" (id 1) (at 21.59 57.15 0))
+    (property "Footprint" "" (id 2) (at 21.59 52.07 0)
+      (effects (font (size 1.27 1.27)) hide)
+    )
+    (property "Datasheet" "" (id 3) (at 21.59 52.07 0)
       (effects (font (size 1.27 1.27)) hide)
     )
@@
     (pin "1")
   )
-  (symbol (lib_name "BZT52C3V3S_1") (lib_id "RP2040-Decoder_Additional_Symbols:BZT52C3V3S") (at 33.02 46.99 270) (unit 1)
-    (in_bom yes) (on_board yes)
-    (property "Reference" "D3" (id 0) (at 27.94 45.72 90)
-      (effects (font (size 1.27 1.27)) (justify left))
-    )
-    (property "Value" "BZT52C3V3S" (id 1) (at 19.05 48.26 90)
-      (effects (font (size 1.27 1.27)) (justify left))
-    )
-    (property "Footprint" "Diode_SMD:D_SOD-323" (id 2) (at 28.575 46.99 0)
-      (effects (font (size 1.27 1.27)) hide)
-    )
-    (property "Datasheet" "https://datasheet.lcsc.com/lcsc/2109071430_YONGYUTAI-BZT52C3V3S_C2892655.pdf" (id 3) (at 26.67 46.99 0)
-      (effects (font (size 1.27 1.27)) hide)
-    )
+  (symbol (lib_name "BZT52C3V3S_1") (lib_id "RP2040-Decoder_Additional_Symbols:BZT52C3V3S") (at 33.02 46.99 90) (mirror x) (unit 1)
+    (in_bom yes) (on_board yes)
+    (property "Reference" "D3" (id 0) (at 38.1 45.72 90)
+      (effects (font (size 1.27 1.27)) (justify left))
+    )
+    (property "Value" "BZT52C3V3S" (id 1) (at 46.99 48.26 90)
+      (effects (font (size 1.27 1.27)) (justify left))
+    )
+    (property "Footprint" "Diode_SMD:D_SOD-323" (id 2) (at 37.465 46.99 0)
+      (effects (font (size 1.27 1.27)) hide)
+    )
+    (property "Datasheet" "https://datasheet.lcsc.com/lcsc/2109071430_YONGYUTAI-BZT52C3V3S_C2892655.pdf" (id 3) (at 39.37 46.99 0)
+      (effects (font (size 1.27 1.27)) hide)
+    )

Commit message: Slight changes to schematic & progress on PCB design
Connections:
- net ADC_EMF_A: now also U4.39 (GPIO27_ADC1)
- net ADC_EMF_B: now also U4.40 (GPIO28_ADC2), U4.41 (GPIO29_ADC3); no longer U4.39 (GPIO27_ADC1)
- net GPIO22: now also U2.7 (INB); no longer U2.6 (INA)
- net GPIO23: now also U2.6 (INA); no longer U2.7 (INB)
- net GPIO24: now also U4.37 (GPIO25); no longer U4.36 (GPIO24)
- no-connect marks 21 -> 19

Commit message: removed 47k resistor
Parts:
- removed R2: 47k, Resistor_SMD:R_0603_1608Metric, symbol Device:R
Changed lines of the file:
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@@
-    (stroke (width 0) (type default) (color 0 0 0 0))
-  )
-  (wire (pts (xy 21.59 41.91) (xy 33.02 41.91))
     (stroke (width 0) (type default) (color 0 0 0 0))
   )
@@
     (stroke (width 0) (type default) (color 0 0 0 0))
   )
-  (wire (pts (xy 21.59 43.18) (xy 21.59 41.91))
-    (stroke (width 0) (type default) (color 0 0 0 0))
-  )
   (wire (pts (xy 199.39 111.76) (xy 220.98 111.76))
     (stroke (width 0) (type default) (color 0 0 0 0))
@@
     (stroke (width 0) (type default) (color 0 0 0 0))
   )
-  (wire (pts (xy 33.02 41.91) (xy 44.45 41.91))
+  (wire (pts (xy 20.32 41.91) (xy 33.02 41.91))
     (stroke (width 0) (type default) (color 0 0 0 0))
   )
@@
   )
   (wire (pts (xy 33.02 52.07) (xy 33.02 50.8))
-    (stroke (width 0) (type default) (color 0 0 0 0))
-  )
-  (wire (pts (xy 21.59 50.8) (xy 21.59 52.07))
     (stroke (width 0) (type default) (color 0 0 0 0))
   )
@@
     (effects (font (size 1.27 1.27)) (justify right bottom))
   )
-  (label "GPIO24" (at 44.45 41.91 180)
-    (effects (font (size 1.27 1.27)) (justify right bottom))
+  (label "GPIO24" (at 20.32 41.91 0)
+    (effects (font (size 1.27 1.27)) (justify left bottom))
   )
   (label "GPIO21" (at 245.11 39.37 0)
@@
     )
     (property "Datasheet" "~" (id 3) (at 81.28 35.56 0)
-      (effects (font (size 1.27 1.27)) hide)
-    )
-    (pin "1")
-    (pin "2")
-  )
-  (symbol (lib_id "Device:R") (at 21.59 46.99 180) (unit 1)
-    (in_bom yes) (on_board yes)
-    (property "Reference" "R2" (id 0) (at 25.4 45.72 0))
-    (property "Value" "47k" (id 1) (at 25.4 48.26 0))
-    (property "Footprint" "Resistor_SMD:R_0603_1608Metric" (id 2) (at 23.368 46.99 90)
-      (effects (font (size 1.27 1.27)) hide)
-    )
-    (property "Datasheet" "~" (id 3) (at 21.59 46.99 0)
       (effects (font (size 1.27 1.27)) hide)
     )
@@
     (pin "1")
   )
-  (symbol (lib_id "power:GND") (at 21.59 52.07 0) (mirror y) (unit 1)
-    (in_bom yes) (on_board yes) (fields_autoplaced)
-    (property "Reference" "#PWR010" (id 0) (at 21.59 58.42 0)
-      (effects (font (size 1.27 1.27)) hide)
-    )
-    (property "Value" "GND" (id 1) (at 21.59 57.15 0))
-    (property "Footprint" "" (id 2) (at 21.59 52.07 0)
-      (effects (font (size 1.27 1.27)) hide)
-    )
-    (property "Datasheet" "" (id 3) (at 21.59 52.07 0)
-      (effects (font (size 1.27 1.27)) hide)
-    )
-    (pin "1")
-  )
   (symbol (lib_id "power:+3V3") (at 22.86 101.6 0) (mirror y) (unit 1)
     (in_bom yes) (on_board yes)
@@
       (reference "#PWR09") (unit 1) (value "GND") (footprint "")
     )
-    (path "/b6343ece-526c-457c-889b-de4a68cd141c"
-      (reference "#PWR010") (unit 1) (value "GND") (footprint "")
-    )
     (path "/00000000-0000-0000-0000-000061f75ece"
       (reference "#PWR011") (unit 1) (value "+1V1") (footprint "")
@@
       (reference "R1") (unit 1) (value "10k") (footprint "Resistor_SMD:R_0603_1608Metric")
     )
-    (path "/00000000-0000-0000-0000-0000621da732"
-      (reference "R2") (unit 1) (value "47k") (footprint "Resistor_SMD:R_0603_1608Metric")
-    )
     (path "/b8f41645-564e-4e6d-89bf-38ca4d783693"

Commit message: - Changes to sorting in measure() function - Changes to Zener Voltage Correction /  measure now returns value in volts - Changes to Motor control - Resistor values changed - Created BOM
Parts:
- R1, R5, R6, R7, R8: value 10k -> 3k9
Changed lines of the file:
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@@
     (in_bom yes) (on_board yes)
     (property "Reference" "R1" (id 0) (at 36.83 25.4 0))
-    (property "Value" "10k" (id 1) (at 36.83 27.94 0))
+    (property "Value" "3k9" (id 1) (at 36.83 27.94 0))
     (property "Footprint" "Resistor_SMD:R_0603_1608Metric" (id 2) (at 34.798 26.67 90)
       (effects (font (size 1.27 1.27)) hide)
@@
     (in_bom yes) (on_board yes)
     (property "Reference" "R6" (id 0) (at 250.19 115.57 0))
-    (property "Value" "10k" (id 1) (at 250.19 118.11 0))
+    (property "Value" "3k9" (id 1) (at 250.19 118.11 0))
     (property "Footprint" "Resistor_SMD:R_0603_1608Metric" (id 2) (at 248.158 116.84 90)
       (effects (font (size 1.27 1.27)) hide)
@@
     (in_bom yes) (on_board yes)
     (property "Reference" "R8" (id 0) (at 250.19 125.73 0))
-    (property "Value" "10k" (id 1) (at 250.19 128.27 0))
+    (property "Value" "3k9" (id 1) (at 250.19 128.27 0))
     (property "Footprint" "Resistor_SMD:R_0603_1608Metric" (id 2) (at 248.158 127 90)
       (effects (font (size 1.27 1.27)) hide)
@@
     (in_bom yes) (on_board yes)
     (property "Reference" "R7" (id 0) (at 217.17 125.73 0))
-    (property "Value" "10k" (id 1) (at 217.17 128.27 0))
+    (property "Value" "3k9" (id 1) (at 217.17 128.27 0))
     (property "Footprint" "Resistor_SMD:R_0603_1608Metric" (id 2) (at 222.758 127 90)
       (effects (font (size 1.27 1.27)) hide)
@@
     (in_bom yes) (on_board yes)
     (property "Reference" "R5" (id 0) (at 217.17 115.57 0))
-    (property "Value" "10k" (id 1) (at 217.17 118.11 0))
+    (property "Value" "3k9" (id 1) (at 217.17 118.11 0))
     (property "Footprint" "Resistor_SMD:R_0603_1608Metric" (id 2) (at 222.758 116.84 90)
       (effects (font (size 1.27 1.27)) hide)
@@
     )
     (path "/00000000-0000-0000-0000-0000621db99e"
-      (reference "R1") (unit 1) (value "10k") (footprint "Resistor_SMD:R_0603_1608Metric")
+      (reference "R1") (unit 1) (value "3k9") (footprint "Resistor_SMD:R_0603_1608Metric")
     )
     (path "/b8f41645-564e-4e6d-89bf-38ca4d783693"
@@
     )
     (path "/00000000-0000-0000-0000-0000623ce830"
-      (reference "R5") (unit 1) (value "10k") (footprint "Resistor_SMD:R_0603_1608Metric")
+      (reference "R5") (unit 1) (value "3k9") (footprint "Resistor_SMD:R_0603_1608Metric")
     )
     (path "/00000000-0000-0000-0000-0000623b9b34"
-      (reference "R6") (unit 1) (value "10k") (footprint "Resistor_SMD:R_0603_1608Metric")
+      (reference "R6") (unit 1) (value "3k9") (footprint "Resistor_SMD:R_0603_1608Metric")
     )
     (path "/00000000-0000-0000-0000-0000623ce82a"
-      (reference "R7") (unit 1) (value "10k") (footprint "Resistor_SMD:R_0603_1608Metric")
+      (reference "R7") (unit 1) (value "3k9") (footprint "Resistor_SMD:R_0603_1608Metric")
     )
     (path "/00000000-0000-0000-0000-0000623ba784"
-      (reference "R8") (unit 1) (value "10k") (footprint "Resistor_SMD:R_0603_1608Metric")
+      (reference "R8") (unit 1) (value "3k9") (footprint "Resistor_SMD:R_0603_1608Metric")
     )
     (path "/00000000-0000-0000-0000-0000620f5623"

Commit message: Finished Board
Parts:
- removed D2: 1N4148WS, Diode_SMD:D_SOD-323, symbol Diode:1N4148WS
- removed D3, D4, D5: BZT52C3V3S, Diode_SMD:D_SOD-323, symbol RP2040-Decoder_Additional_Symbols:BZT52C3V3S
- removed J1: DCC_IN, Connector_PinHeader_1.00mm:PinHeader_1x02_P1.00mm_Vertical, symbol Connector:Conn_01x02_Male
- removed J2: MOTOR_CONN, Connector_PinHeader_1.00mm:PinHeader_1x04_P1.00mm_Vertical, symbol Connector:Conn_01x04_Male
- removed J3: GPIO_CONN, Connector_PinHeader_1.00mm:PinHeader_1x06_P1.00mm_Vertical, symbol Connector:Conn_01x06_Male
- removed J4: DEBUG_CONN, Connector_PinHeader_1.00mm:PinHeader_1x04_P1.00mm_Vertical, symbol Connector:Conn_01x04_Male
- removed Q1, Q2, Q3, Q4: WNM2030, RP2040-Decoder_Additional_Footprints:SOT-723-Extended_Pad, symbol RP2040-Decoder_Additional_Symbols:WNM2030
- added J1: T0, TestPoint:TestPoint_Pad_D2.0mm, symbol Connector:Conn_01x01_Male
- added J10, J5: 2, TestPoint:TestPoint_Pad_D2.0mm, symbol Connector:Conn_01x01_Male
- added J11, J6: 3, TestPoint:TestPoint_Pad_D2.0mm, symbol Connector:Conn_01x01_Male
- added J12: 4, TestPoint:TestPoint_Pad_D2.0mm, symbol Connector:Conn_01x01_Male
- added J13: 5, TestPoint:TestPoint_Pad_D2.0mm, symbol Connector:Conn_01x01_Male
- added J14: +V, TestPoint:TestPoint_Pad_D2.0mm, symbol Connector:Conn_01x01_Male
- added J15: M_OUT_B, TestPoint:TestPoint_Pad_D2.0mm, symbol Connector:Conn_01x01_Male
- added J16: M_OUT_A, TestPoint:TestPoint_Pad_D2.0mm, symbol Connector:Conn_01x01_Male
- added J17: GND, TestPoint:TestPoint_Pad_D2.0mm, symbol Connector:Conn_01x01_Male
- added J18: SWCLK, TestPoint:TestPoint_Pad_D2.0mm, symbol Connector:Conn_01x01_Male
- added J19: SWDIO, TestPoint:TestPoint_Pad_D2.0mm, symbol Connector:Conn_01x01_Male
- added J2: T1, TestPoint:TestPoint_Pad_D2.0mm, symbol Connector:Conn_01x01_Male
- added J20: RUN, TestPoint:TestPoint_Pad_D2.0mm, symbol Connector:Conn_01x01_Male
- added J3, J8: 0, TestPoint:TestPoint_Pad_D2.0mm, symbol Connector:Conn_01x01_Male
- added J4, J9: 1, TestPoint:TestPoint_Pad_D2.0mm, symbol Connector:Conn_01x01_Male
- added J7: +3V3, TestPoint:TestPoint_Pad_D2.0mm, symbol Connector:Conn_01x01_Male
- added Q1, Q2, Q3, Q4, Q5: T2N7002BK, Package_TO_SOT_SMD:SOT-23, symbol RP2040-Decoder_Additional_Symbols:T2N7002BK
- added R2: 6k8, RP2040-Decoder_Additional_Footprints:R_0603_1608Metric, symbol Device:R
- C1, C10, C11, C12, C13, C15, C16, C17, C2, C3, C4, C7, C8, C9: footprint Capacitor_SMD:C_0603_1608Metric -> RP2040-Decoder_Additional_Footprints:C_0603_1608Metric
- C14, C5, C6: value 2u2 -> 10u; footprint Capacitor_SMD:C_0603_1608Metric -> RP2040-Decoder_Additional_Footprints:C_0603_1608Metric
- R1, R5, R6: value 3k9 -> 6k8; footprint Resistor_SMD:R_0603_1608Metric -> RP2040-Decoder_Additional_Footprints:R_0603_1608Metric
- R3, R4, R9: footprint Resistor_SMD:R_0603_1608Metric -> RP2040-Decoder_Additional_Footprints:R_0603_1608Metric
- R7, R8: value 3k9 -> 1k; footprint Resistor_SMD:R_0603_1608Metric -> RP2040-Decoder_Additional_Footprints:R_0603_1608Metric
- U2: footprint Package_SO:SOIC-8-1EP_3.9x4.9mm_P1.27mm_EP2.41x3.3mm_ThermalVias -> RP2040-Decoder_Additional_Footprints:SOIC-8-1EP_3.9x4.9mm_P1.27mm_EP2.41x3.3mm_ThermalVias
- U3: footprint Package_SO:SOIC-8_5.23x5.23mm_P1.27mm -> RP2040-Decoder_Additional_Footprints:SOIC-8_5.23x5.23mm_P1.27mm
Connections:
- net +3V3: now also J7.1 (Pin_1)
- net ADC_EMF_A: no longer U4.39 (GPIO27_ADC1)
- net ADC_EMF_B: now also U4.39 (GPIO27_ADC1); no longer U4.40 (GPIO28_ADC2), U4.41 (GPIO29_ADC3)
- net GND: now also J17.1 (Pin_1), Q1.2 (S), Q2.2 (S), Q3.2 (S), Q4.2 (S), Q5.2 (S), R2.1
- net GPIO18: now also Q2.1 (G)
- net GPIO19: now also Q3.1 (G)
- net GPIO20: now also Q4.1 (G)
- net GPIO21: now also Q5.1 (G)
- net GPIO24: now also Q1.3 (D)
- net MOTOR_OUT_A: now also J15.1 (Pin_1)
- net MOTOR_OUT_B: now also J16.1 (Pin_1)
- net at R1.1: now also Q1.1 (G), R2.2
- net at R1.2: now also D1.1, J1.1 (Pin_1); no longer D1.2
- net at U4.7 (GPIO5): now also J13.1 (Pin_1)
- net at U4.6 (GPIO4): now also J12.1 (Pin_1)
- net at U4.5 (GPIO3): now also J11.1 (Pin_1)
- net at U4.4 (GPIO2): now also J10.1 (Pin_1)
- net at U4.3 (GPIO1): now also J9.1 (Pin_1)
- net at U4.2 (GPIO0): now also J8.1 (Pin_1)
- net at U4.26 (RUN): now also J20.1 (Pin_1)
- net at U4.25 (SWD): now also J19.1 (Pin_1)
- net at U4.24 (SWCLK): now also J18.1 (Pin_1)
- net +12V renamed +V
- net +V: now also J14.1 (Pin_1)
- new net: J5.1 (Pin_1), Q4.3 (D)
- new net: D1.2, J2.1 (Pin_1)
- new net: J3.1 (Pin_1), Q2.3 (D)
- new net: J6.1 (Pin_1), Q5.3 (D)
- new net: J4.1 (Pin_1), Q3.3 (D)
- no-connect marks 19 -> 17
Other:
- note added: "GPIO24 is pulled up in RP2040"
- note added: "Gate GPIOs are pulled down in RP2040"
- moved on the sheet: C1, C16, C17, C2, D1, U1

Commit message: small changes to schematic and update to docs/svg
Other:
- note added: "Gates are pulled down using RP2040 pull-down resistors"
- note removed: "Gate GPIOs are pulled down in RP2040"
- moved on the sheet: J18, J19, J20
