File: KiCad/RP2040-Decoder.kicad_pcb (KiCad board)
At the start: 2 copper layers, 25 x 20 mm, 57 parts, among them J1 T0, J10 2, J11 3, J12 4, J13 5, J14 +V, J15 M_OUT_B, J16 M_OUT_A, J17 GND, J18 SWCLK, J19 SWDIO, J2 T1, J20 RUN, J3 0, J4 1, J5 2, J6 3, J7 +3V3, J8 0, J9 1, Q1 T2N7002BK, U1 PJ75AL33SA, U2 BDR6133, U3 W25Q64JVSSIQ, U4 RP2040, Y1 X322512MSB4SI

Commit message: AUX GPIO are now 24-27, ADC GPIO are now 28 and 29 DCC_IN is now 21 - Board Revision is now "0.3" - Omitted Rev. in Kicad filenames
Parts:
- Q2: renamed from Q 2
- Q3: renamed from Q 3
- Q4: renamed from Q 4
- Q5: renamed from Q 5
- moved C9 0.87 mm to (149.1, 105.3)
- moved C8 0.18 mm to (148.9, 101.2)
- moved C14 0.15 mm to (148.9, 99.8)
Connections:
- C17 pad 1: Net-(C17-Pad1) -> Net-(R9-Pad2)
- Q1 pad 3: /GPIO24 -> /GPIO21
- Q2 pad 1: /GPIO18 -> /GPIO24
- Q3 pad 1: /GPIO19 -> /GPIO25
- Q4 pad 1: /GPIO20 -> /GPIO26
- Q5 pad 1: /GPIO21 -> /GPIO27
- R9 pad 2: GND -> Net-(R9-Pad2)
- U4 pad 29: /GPIO18 -> unconnected-(U4-Pad29)
- U4 pad 30: /GPIO19 -> unconnected-(U4-Pad30)
- U4 pad 31: /GPIO20 -> unconnected-(U4-Pad31)
- U4 pad 36: unconnected-(U4-Pad36) -> /GPIO24
- U4 pad 37: /GPIO24 -> /GPIO25
- U4 pad 38: /ADC_EMF_A -> /GPIO26
- U4 pad 39: /ADC_EMF_B -> /GPIO27
- U4 pad 40: unconnected-(U4-Pad40) -> /ADC_EMF_A
- U4 pad 41: unconnected-(U4-Pad41) -> /ADC_EMF_B
- Y1 pad 1: Net-(C17-Pad1) -> Net-(R9-Pad2)
Routing:
- net Net-(R9-Pad2): track 0.00 -> 20.3 mm, vias 0 -> 2
- net /GPIO25: track 0.00 -> 14.6 mm
- net /GPIO26: track 0.00 -> 13.8 mm
- net /GPIO20: track 13.6 -> 0.00 mm
- net /GPIO19: track 13.4 -> 0.00 mm
- net /GPIO21: track 9.58 -> 20.5 mm, vias 0 -> 4
- net /GPIO27: track 0.00 -> 9.63 mm
- net /GPIO18: track 9.39 -> 0.00 mm
- net /GPIO24: track 17.2 -> 11.0 mm, vias 2 -> 0
- net Net-(C17-Pad1): track 1.83 -> 0.00 mm
- net Net-(U4-Pad20): track 10.8 -> 9.37 mm
- net /GPIO22: track 18.8 -> 19.5 mm, vias 0 -> 2
- net Net-(D1-Pad1): track 28.5 -> 27.9 mm
- net +3V3: track 93.2 -> 92.6 mm
- net /GPIO23: track 17.8 -> 17.9 mm, vias 0 -> 2
Other:
- board text added: "Rev. 0.3"
- board text removed: "Rev. 0.2"

Commit message: Add note regarding U1 / PJ75AL33SA LDO / Issue 23 to schematic; Update KiCad Project to version 7; Change C16 and C17 to 10pF
Parts:
- C16, C17: value 33p -> 10p

Commit message: Replace PJ75AL33SA with HT7533S
Parts:
- U1: value PJ75AL33SA -> HT7533S
Changed lines of the file:
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@@
     (property "Sheetname" "")
     (attr smd)
-    (fp_text reference "U1" (at 2.3 0 180) (layer "F.SilkS")
+    (fp_text reference "U1" (at 2.3 0) (layer "F.SilkS")
         (effects (font (size 1 1) (thickness 0.15)))
     )
-    (fp_text value "PJ75AL33SA" (at -1.1 0 180) (layer "F.Fab")
+    (fp_text value "HT7533S" (at -1.1 0) (layer "F.Fab")
         (effects (font (size 0.3 0.3) (thickness 0.05)))
     )
