File: KiCad/RP2040-Decoder.kicad_pcb (KiCad board)
At the start: 4 copper layers, 25 x 20 mm, 68 parts, among them J1 Conn_01x01, J10 Conn_01x01, J11 Conn_01x01, J12 Conn_01x01, J13 Conn_01x01, J14 Conn_01x01, J15 Conn_01x01, J16 Conn_01x01, J17 Conn_01x01, J18 Conn_01x01, J19 Conn_01x01, J2 Conn_01x01, J20 Conn_01x01, J21 Conn_01x01, J3 USB_C_Receptacle_USB2.0_16P, J4 Conn_01x01, J5 Conn_01x01, J6 Conn_01x01, J7 Conn_01x01, J8 Conn_01x01, J9 Conn_01x01, Q1 Si1308EDL, Q2 Si1308EDL, Q3 Si1308EDL, Q4 Si1308EDL, Q5 Si1308EDL, U1 MIC5200-3.3YS, U2 W25Q64JVSSIQ, U3 RP2040, U4 BDR6133, Y1 X322512MSB4SI

Commit message: Add LCSC Part numbers
Parts:
- R2, R3: value 5k11 -> 5k1

Commit message: Update Docs; Add 3D-Models for flash and Motor driver; Update Readme; Check program code for exceeding size in CMakeLists.txt; Moved measure() function to core1.c/core1.h; Added direction enum typedef; Update Control Loop Block Diagram;
Parts:
- U2: footprint Package_SO:SOIC-8_5.23x5.23mm_P1.27mm -> RP2040-Decoder_Additional_Footprints:SOIC-8_5.23x5.23mm_P1.27mm
- U4: footprint Package_SO:SOIC-8-1EP_3.9x4.9mm_P1.27mm_EP2.41x3.3mm_ThermalVias -> RP2040-Decoder_Additional_Footprints:SOIC-8-1EP_3.9x4.9mm_P1.27mm_EP2.41x3.3mm_ThermalVias
Changed lines of the file:
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@@
 		)
 	)
-	(footprint "Package_SO:SOIC-8-1EP_3.9x4.9mm_P1.27mm_EP2.41x3.3mm_ThermalVias"
+	(footprint "RP2040-Decoder_Additional_Footprints:SOIC-8-1EP_3.9x4.9mm_P1.27mm_EP2.41x3.3mm_ThermalVias"
 		(layer "F.Cu")
 		(at 159.8 93.9 -90)
@@
 		(tags "SOIC SO")
 		(property "Reference" "U4"
-			(at -1.4 6.7 180)
+			(at -0.2 -4.3 -90)
 			(layer "F.SilkS")
-			(hide yes)
 			(effects
 				(font
@@
 		)
 		(property "Value" "BDR6133"
-			(at 0 3.4 90)
+			(at 0 3.4 -90)
 			(layer "F.Fab")
-			(hide yes)
 			(effects
 				(font
@@
 			)
 		)
-		(property "Footprint" "Package_SO:SOIC-8-1EP_3.9x4.9mm_P1.27mm_EP2.41x3.3mm_ThermalVias"
-			(at 0 0 90)
+		(property "Footprint" "RP2040-Decoder_Additional_Footprints:SOIC-8-1EP_3.9x4.9mm_P1.27mm_EP2.41x3.3mm_ThermalVias"
+			(at 0 0 -90)
 			(layer "F.Fab")
 			(hide yes)
@@
 			)
 		)
-		(property "Datasheet" "https://datasheet.lcsc.com/lcsc/2101211904_Bardeen-Micro--BDR6133_C2687793.pdf"
-			(at 0 0 90)
+		(property "Datasheet" "https://www.lcsc.com/datasheet/lcsc_datasheet_2409291808_Bardeen-Micro--BDR6133_C2687793.pdf"
+			(at 0 0 -90)
 			(layer "F.Fab")
 			(hide yes)
@@
 			)
 		)
-		(property "Description" ""
-			(at 0 0 90)
+		(property "Description" "H-Bridge driver, 2.8A, 2V to 24V, PWM input, ESOP8"
+			(at 0 0 -90)
 			(layer "F.Fab")
 			(hide yes)
@@
 			)
 		)
-		(property ki_fp_filters "WSON*1EP*2x2mm*P0.5mm*")
+		(property ki_fp_filters "SOIC-8-1EP_3.9x4.9mm_P1.27mm_EP2.29x3mm")
 		(sheetname "Root")
 		(sheetfile "RP2040-Decoder.kicad_sch")
 		(attr smd)
 		(fp_line
-			(start 0 2.56)
-			(end -1.95 2.56)
+			(start -1.55 2.56)
+			(end -3.4 2.56)
 			(stroke
 				(width 0.12)
@@
 		)
 		(fp_line
-			(start 0 2.56)
-			(end 1.95 2.56)
+			(start 1.55 2.56)
+			(end 3.4 2.56)
 			(stroke
 				(width 0.12)
@@
 		)
 		(fp_line
-			(start 0 -2.56)
-			(end -1.95 -2.56)
+			(start -1.55 -2.56)
+			(end -3.4 -2.56)
 			(stroke
 				(width 0.12)
@@
 		)
 		(fp_line
-			(start 0 -2.56)
-			(end 1.95 -2.56)
-			(stroke
-				(width 0.12)
-				(type solid)
-			)
-			(layer "F.SilkS")
-		)
-		(fp_poly
-			(pts
-				(xy -2.7 -2.465) (xy -2.94 -2.795) (xy -2.46 -2.795) (xy -2.7 -2.465)
-			)
+			(start 1.55 -2.56)
+			(end 3.4 -2.56)
 			(stroke
 				(width 0.12)
 				(type solid)
 			)
-			(fill solid)
 			(layer "F.SilkS")
 		)
@@
 		)
 		(fp_text user "${REFERENCE}"
-			(at 0 0 180)
+			(at 0 0 -90)
 			(layer "F.Fab")
 			(effects
@@
 		(pad "9" thru_hole circle
 			(at -0.7 -1.2 270)
-			(size 0.4 0.4)
-			(drill 0.3)
-			(property pad_prop_heatsink)
-			(layers "*.Cu" "Dwgs.User")
+			(size 0.5 0.5)
+			(drill 0.2)
+			(layers "*.Cu")
 			(remove_unused_layers no)
 			(net 4 "GND")
@@
 		(pad "9" thru_hole circle
 			(at -0.7 0 270)
-			(size 0.4 0.4)
-			(drill 0.3)
-			(property pad_prop_heatsink)
+			(size 0.5 0.5)
+			(drill 0.2)
 			(layers "*.Cu")
 			(remove_unused_layers no)
@@
 		(pad "9" thru_hole circle
 			(at -0.7 1.2 270)
-			(size 0.4 0.4)
-			(drill 0.3)
-			(property pad_prop_heatsink)
+			(size 0.5 0.5)
+			(drill 0.2)
 			(layers "*.Cu")
 			(remove_unused_layers no)
@@
 			(at 0 0 270)
 			(size 1.9 2.9)
-			(property pad_prop_heatsink)
 			(layers "B.Cu")
 			(net 4 "GND")
 			(pinfunction "GND")
 			(pintype "passive")
-			(zone_connect 2)
 		)
 		(pad "9" smd rect
 			(at 0 0 270)
 			(size 2.41 3.3)
-			(property pad_prop_heatsink)
 			(layers "F.Cu" "F.Mask")
 			(net 4 "GND")
 			(pinfunction "GND")
 			(pintype "passive")
-			(zone_connect 2)
 		)
 		(pad "9" thru_hole circle
 			(at 0.7 -1.2 270)
-			(size 0.4 0.4)
-			(drill 0.3)
-			(property pad_prop_heatsink)
+			(size 0.5 0.5)
+			(drill 0.2)
 			(layers "*.Cu")
 			(remove_unused_layers no)
@@
 		(pad "9" thru_hole circle
 			(at 0.7 0 270)
-			(size 0.4 0.4)
-			(drill 0.3)
-			(property pad_prop_heatsink)
+			(size 0.5 0.5)
+			(drill 0.2)
 			(layers "*.Cu")
 			(remove_unused_layers no)
@@
 		(pad "9" thru_hole circle
 			(at 0.7 1.2 270)
-			(size 0.4 0.4)
-			(drill 0.3)
-			(property pad_prop_heatsink)
+			(size 0.5 0.5)
+			(drill 0.2)
 			(layers "*.Cu")
 			(remove_unused_layers no)
@@
 			(pintype "passive")
 		)
-		(model "${KICAD8_3DMODEL_DIR}/Package_SO.3dshapes/SOIC-8-1EP_3.9x4.9mm_P1.27mm_EP2.41x3.3mm.wrl"
+		(model "${KICAD8_3DMODEL_DIR}/Package_SO.3dshapes/SOIC-8_3.9x4.9mm_P1.27mm.wrl"
 			(offset
 				(xyz 0 0 0)
@@
 		)
 	)
-	(footprint "Package_SO:SOIC-8_5.23x5.23mm_P1.27mm"
+	(footprint "RP2040-Decoder_Additional_Footprints:SOIC-8_5.23x5.23mm_P1.27mm"
 		(layer "F.Cu")
 		(at 142.1 92.8 180)
@@
 		(tags "SOIC SO")
 		(property "Reference" "U2"
-			(at 1 -3.5 0)
+			(at 0 -3.56 180)
 			(layer "F.SilkS")
 			(effects
@@
 		)
 		(property "Value" "W25Q64JVSSIQ"
-			(at 0 3.56 0)
+			(at 0 3.56 180)
 			(layer "F.Fab")
-			(hide yes)
 			(effects
 				(font
@@
 			)
 		)
-		(property "Footprint" "Package_SO:SOIC-8_5.23x5.23mm_P1.27mm"
-			(at 0 0 0)
+		(property "Footprint" "RP2040-Decoder_Additional_Footprints:SOIC-8_5.23x5.23mm_P1.27mm"
+			(at 0 0 180)
 			(layer "F.Fab")
 			(hide yes)
@@
 		)
 		(property "Datasheet" "https://www.winbond.com/resource-files/w25q64jv%20revj%2003272018%20plus.pdf"
-			(at 0 0 0)
+			(at 0 0 180)
 			(layer "F.Fab")
 			(hide yes)
@@
 		)
 		(property "Description" ""
-			(at 0 0 0)
+			(at 0 0 180)
 			(layer "F.Fab")
 			(hide yes)
@@
 		)
 		(fp_line
-			(start -2.725 -2.725)
-			(end -2.725 -2.465)
+			(start -2.725 -2.465)
+			(end -4.4 -2.465)
 			(stroke
 				(width 0.12)
@@
 			(layer "F.SilkS")
 		)
-		(fp_poly
-			(pts
-				(xy -3.5075 -2.465) (xy -3.7475 -2.795) (xy -3.2675 -2.795) (xy -3.5075 -2.465)
-			)
+		(fp_line
+			(start -2.725 -2.725)
+			(end -2.725 -2.465)
 			(stroke
 				(width 0.12)
 				(type solid)
 			)
-			(fill solid)
 			(layer "F.SilkS")
 		)
@@
 		)
 		(fp_text user "${REFERENCE}"
-			(at 0 0 0)
+			(at 0 0 180)
 			(layer "F.Fab")
 			(effects
@@
 			(pintype "power_in")
 		)
-		(model "${KICAD8_3DMODEL_DIR}/Package_SO.3dshapes/SOIC-8_5.23x5.23mm_P1.27mm.wrl"
+		(model "${KICAD8_3DMODEL_DIR}/Package_SO.3dshapes/SOIC-8_5.275x5.275mm_P1.27mm.wrl"
 			(offset
 				(xyz 0 0 0)
