File: KiCad/RP2040-Decoder.kicad_sch (KiCad schematic)
At the start: 57 parts, among them J1 T0, J10 2, J11 3, J12 4, J13 5, J14 +V, J15 M_OUT_B, J16 M_OUT_A, J17 GND, J18 SWCLK, J19 SWDIO, J2 T1, J20 RUN, J3 0, J4 1, J5 2, J6 3, J7 +3V3, J8 0, J9 1, Q1 T2N7002BK, Q2 T2N7002BK, Q3 T2N7002BK, Q4 T2N7002BK, Q5 T2N7002BK, U1 PJ75AL33SA, U2 BDR6133, U3 W25Q64JVSSIQ, U4 RP2040, Y1 X322512MSB4SI

Commit message: AUX GPIO are now 24-27, ADC GPIO are now 28 and 29 DCC_IN is now 21 - Board Revision is now "0.3" - Omitted Rev. in Kicad filenames
Connections:
- net ADC_EMF_A: now also U4.40 (GPIO28_ADC2); no longer U4.38 (GPIO26_ADC0)
- net ADC_EMF_B: now also U4.41 (GPIO29_ADC3); no longer U4.39 (GPIO27_ADC1)
- net GND: no longer R9.2
- net GPIO21: now also Q1.3 (D); no longer Q5.1 (G)
- net GPIO24: now also Q2.1 (G), U4.36 (GPIO24); no longer Q1.3 (D), U4.37 (GPIO25)
- net at C17.1, Y1.1: now also R9.2
- net GPIO18: no longer names the net of U4.29 (GPIO18)
- net GPIO18: no longer Q2.1 (G)
- net GPIO19: no longer names the net of U4.30 (GPIO19)
- net GPIO19: no longer Q3.1 (G)
- net GPIO20: no longer names the net of U4.31 (GPIO20)
- net GPIO20: no longer Q4.1 (G)
- new net GPIO25: Q3.1 (G), U4.37 (GPIO25)
- new net GPIO26: Q4.1 (G), U4.38 (GPIO26_ADC0)
- new net GPIO27: Q5.1 (G), U4.39 (GPIO27_ADC1)
Other:
- note added: "GPIO21 is pulled up internally in RP2040"
- note removed: "GPIO24 is pulled up in RP2040"
- moved on the sheet: C16, C17, R9, Y1

Commit message: working on PCB
looking to mimic RPi's own minimal PCB
Parts:
- removed C9: 100n, RP2040-Decoder_Additional_Footprints:C_0603_1608Metric, symbol Device:C
- C1, C14, C16, C17, C2: footprint RP2040-Decoder_Additional_Footprints:C_0603_1608Metric -> Capacitor_SMD:C_0603_1608Metric
- C10, C11, C12, C13, C15, C3, C4, C7, C8: footprint RP2040-Decoder_Additional_Footprints:C_0603_1608Metric -> Capacitor_SMD:C_0402_1005Metric
- C5, C6: value 10u -> 1u; footprint RP2040-Decoder_Additional_Footprints:C_0603_1608Metric -> Capacitor_SMD:C_0402_1005Metric
