File: KiCad/RP2040-Decoder.kicad_sch (KiCad schematic)
At the start: 57 parts, among them J1 T0, J10 2, J11 3, J12 4, J13 5, J14 +V, J15 M_OUT_B, J16 M_OUT_A, J17 GND, J18 SWCLK, J19 SWDIO, J2 T1, J20 RUN, J3 0, J4 1, J5 2, J6 3, J7 +3V3, J8 0, J9 1, Q1 T2N7002BK, Q2 T2N7002BK, Q3 T2N7002BK, Q4 T2N7002BK, Q5 T2N7002BK, U1 PJ75AL33SA, U2 BDR6133, U3 W25Q64JVSSIQ, U4 RP2040, Y1 X322512MSB4SI

Commit message: Add note regarding U1 / PJ75AL33SA LDO / Issue 23 to schematic; Update KiCad Project to version 7; Change C16 and C17 to 10pF
Parts:
- C16, C17: value 33p -> 10p
Other:
- note added: "!"

Commit message: Replace PJ75AL33SA with HT7533S
Parts:
- removed U1: PJ75AL33SA, Package_TO_SOT_SMD:SOT-23, symbol RP2040-Decoder_Additional_Symbols:PJ75AL33SA
- added U1: HT7533S, Package_TO_SOT_SMD:SOT-23, symbol RP2040-Decoder_Additional_Symbols:HT7533S
Connections:
- net +3V3: now also U1.2 (VOUT)
- net +V: now also U1.3 (VIN)
- net GND: now also U1.1 (GND)
Other:
- note removed: "!"
Changed lines of the file:
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@@
     (stroke (width 0) (type default))
-  )
-  (text_box "Please refer to issue #23 regarding U1"
-    (at 49.53 12.7 0) (size 26.67 6.35)
-    (stroke (width 0) (type default))
-    (fill (type none))
-    (effects (font (size 1.5 1.5)) (justify left top))
   )
   (text "Gates are pulled down using\nRP2040 pull-down resistors"
@@
     (effects (font (size 1.27 1.27)) (justify left bottom))
   )
-  (text "!" (at 45.72 17.78 0)
-    (effects (font (size 3.5 3.5) (thickness 0.7) bold (color 255 0 15 1)) (justify left bottom))
-  )
   (text "Motor Driver" (at 201.93 87.63 0)
     (effects (font (size 2.54 2.54)) (justify left bottom))
@@
   (text "Aux Outputs" (at 172.72 24.13 0)
     (effects (font (size 2.54 2.54)) (justify left bottom))
-  )
-  (text "!" (at 80.01 17.78 0)
-    (effects (font (size 3.5 3.5) (thickness 0.7) bold (color 255 0 15 1)) (justify right bottom))
   )
   (text "Crystal Oscillator" (at 26.67 138.43 0)
@@
         (path "/11d18738-0f49-4d63-b61c-22a93efd5959"
           (reference "#PWR019") (unit 1)
+        )
+      )
+    )
+  )
+  (symbol (lib_id "RP2040-Decoder_Additional_Symbols:HT7533S") (at 60.96 30.48 0) (mirror y) (unit 1)
+    (in_bom yes) (on_board yes) (dnp no)
+    (property "Reference" "U1" (at 60.96 24.13 0)
+      (effects (font (size 1.27 1.27)))
+    )
+    (property "Value" "HT7533S" (at 60.96 26.67 0)
+      (effects (font (size 1.27 1.27)))
+    )
+    (property "Footprint" "Package_TO_SOT_SMD:SOT-23" (at 59.69 39.37 0)
+      (effects (font (size 1.27 1.27) italic) hide)
+    )
+    (property "Datasheet" "https://datasheet.lcsc.com/lcsc/2311091732_UMW-Youtai-Semiconductor-Co---Ltd--HT7533S_C347215.pdf" (at 58.42 41.91 0)
+      (effects (font (size 1.27 1.27)) hide)
+    )
+    (pin "3")
+    (pin "2")
+    (pin "1")
+    (instances
+      (project "RP2040-Decoder"
+        (path "/11d18738-0f49-4d63-b61c-22a93efd5959"
+          (reference "U1") (unit 1)
         )
       )
@@
         )
       )
-    )
-  )
-  (symbol (lib_id "RP2040-Decoder_Additional_Symbols:PJ75AL33SA") (at 60.96 30.48 0) (mirror y) (unit 1)
-    (in_bom yes) (on_board yes) (dnp no)
-    (property "Reference" "U1" (at 60.96 24.13 0)
-      (effects (font (size 1.27 1.27)))
-    )
-    (property "Value" "PJ75AL33SA" (at 60.96 26.67 0)
-      (effects (font (size 1.27 1.27)))
-    )
-    (property "Footprint" "Package_TO_SOT_SMD:SOT-23" (at 59.69 39.37 0)
-      (effects (font (size 1.27 1.27) italic) hide)
-    )
-    (property "Datasheet" "https://datasheet.lcsc.com/lcsc/1912111437_PJSEMI-PJ75AL33SA_C411736.pdf" (at 58.42 41.91 0)
-      (effects (font (size 1.27 1.27)) hide)
-    )
-    (pin "1")
-    (pin "2")
-    (pin "3")
-    (instances
-      (project "RP2040-Decoder"
-        (path "/11d18738-0f49-4d63-b61c-22a93efd5959"
-          (reference "U1") (unit 1)
-        )
-      )
