File: KiCad/RP2040-Decoder.kicad_sch (KiCad schematic)
At the start: 68 parts, among them J1 Conn_01x01, J10 Conn_01x01, J11 Conn_01x01, J12 Conn_01x01, J13 Conn_01x01, J14 Conn_01x01, J15 Conn_01x01, J16 Conn_01x01, J17 Conn_01x01, J18 Conn_01x01, J19 Conn_01x01, J2 Conn_01x01, J20 Conn_01x01, J21 Conn_01x01, J3 USB_C_Receptacle_USB2.0_16P, J4 Conn_01x01, J5 Conn_01x01, J6 Conn_01x01, J7 Conn_01x01, J8 Conn_01x01, J9 Conn_01x01, Q1 Si1308EDL, Q2 Si1308EDL, Q3 Si1308EDL, Q4 Si1308EDL, Q5 Si1308EDL, U1 MIC5200-3.3YS, U2 W25Q64JVSSIQ, U3 RP2040, U4 BDR6133, Y1 X322512MSB4SI

Commit message: Add LCSC Part numbers
Parts:
- C1, C4: LCSC Part Number (none) -> C32949
- C10, C11, C12, C14, C15, C16, C2, C6, C7: LCSC Part Number (none) -> C1525
- C13, C18, C8, C9: LCSC Part Number (none) -> C15525
- C17, C3, C5: LCSC Part Number (none) -> C96446
- D1: LCSC Part Number (none) -> C191023
- D2: LCSC Part Number (none) -> C880910
- D3: LCSC Part Number (none) -> C2286
- J3: LCSC Part Number (none) -> C2927038
- Q1, Q2, Q3, Q4, Q5: LCSC Part Number (none) -> C469327
- R1: now not fitted
- R10, R13, R15, R4, R5: LCSC Part Number (none) -> C11702
- R11: LCSC Part Number (none) -> C25087
- R12, R14, R8, R9: LCSC Part Number (none) -> C25917
- R2, R3: value 5k11 -> 5k1; LCSC Part Number (none) -> C25905
- R6, R7: LCSC Part Number (none) -> C138021
- U1: LCSC Part Number (none) -> C5343216
- U2: LCSC Part Number (none) -> C179171
- U3: LCSC Part Number (none) -> C2040
- U4: LCSC Part Number (none) -> C2687793
- Y1: LCSC Part Number (none) -> C9002

Commit message: Changed 'LCSC Part Number' Field to 'LCSC Part #'
Parts:
- C1, C4: LCSC Part # (none) -> C32949; LCSC Part Number C32949 -> (none)
- C10, C11, C12, C14, C15, C16, C2, C6, C7: LCSC Part # (none) -> C1525; LCSC Part Number C1525 -> (none)
- C13, C18, C8, C9: LCSC Part # (none) -> C15525; LCSC Part Number C15525 -> (none)
- C17, C3, C5: LCSC Part # (none) -> C96446; LCSC Part Number C96446 -> (none)
- D1: LCSC Part # (none) -> C191023; LCSC Part Number C191023 -> (none)
- D2: LCSC Part # (none) -> C880910; LCSC Part Number C880910 -> (none)
- D3: LCSC Part # (none) -> C2286; LCSC Part Number C2286 -> (none)
- J3: LCSC Part # (none) -> C2927038; LCSC Part Number C2927038 -> (none)
- Q1, Q2, Q3, Q4, Q5: LCSC Part # (none) -> C469327; LCSC Part Number C469327 -> (none)
- R10, R13, R15, R4, R5: LCSC Part # (none) -> C11702; LCSC Part Number C11702 -> (none)
- R11: LCSC Part # (none) -> C25087; LCSC Part Number C25087 -> (none)
- R12, R14, R8, R9: LCSC Part # (none) -> C25917; LCSC Part Number C25917 -> (none)
- R2, R3: LCSC Part # (none) -> C25905; LCSC Part Number C25905 -> (none)
- R6, R7: LCSC Part # (none) -> C138021; LCSC Part Number C138021 -> (none)
- U1: LCSC Part # (none) -> C5343216; LCSC Part Number C5343216 -> (none)
- U2: LCSC Part # (none) -> C179171; LCSC Part Number C179171 -> (none)
- U3: LCSC Part # (none) -> C2040; LCSC Part Number C2040 -> (none)
- U4: LCSC Part # (none) -> C2687793; LCSC Part Number C2687793 -> (none)
- Y1: LCSC Part # (none) -> C9002; LCSC Part Number C9002 -> (none)

Commit message: Moving some components on the schematic
Parts:
- Q1, Q2, Q3, Q4, Q5: JLCPCB Rotation Offset (none) -> 180
- U3: JLCPCB Rotation Offset (none) -> -90
Other:
- moved on the sheet: C17, C18, J18, J19, J20, J21, J3, R12, R13, R14, R15, R2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

Commit message: Update Docs; Add 3D-Models for flash and Motor driver; Update Readme; Check program code for exceeding size in CMakeLists.txt; Moved measure() function to core1.c/core1.h; Added direction enum typedef; Update Control Loop Block Diagram;
Parts:
- U2: footprint Package_SO:SOIC-8_5.23x5.23mm_P1.27mm -> RP2040-Decoder_Additional_Footprints:SOIC-8_5.23x5.23mm_P1.27mm
- U4: footprint Package_SO:SOIC-8-1EP_3.9x4.9mm_P1.27mm_EP2.41x3.3mm_ThermalVias -> RP2040-Decoder_Additional_Footprints:SOIC-8-1EP_3.9x4.9mm_P1.27mm_EP2.41x3.3mm_ThermalVias
Changed lines of the file:
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@@
 			)
 		)
-		(property "Footprint" "Package_SO:SOIC-8_5.23x5.23mm_P1.27mm"
+		(property "Footprint" "RP2040-Decoder_Additional_Footprints:SOIC-8_5.23x5.23mm_P1.27mm"
 			(at 64.77 142.24 0)
 			(effects
@@
 			)
 		)
-		(property "Footprint" "Package_SO:SOIC-8-1EP_3.9x4.9mm_P1.27mm_EP2.41x3.3mm_ThermalVias"
+		(property "Footprint" "RP2040-Decoder_Additional_Footprints:SOIC-8-1EP_3.9x4.9mm_P1.27mm_EP2.41x3.3mm_ThermalVias"
 			(at 247.65 144.78 0)
 			(effects
@@
 			)
 		)
-		(property "Datasheet" "https://datasheet.lcsc.com/lcsc/2101211904_Bardeen-Micro--BDR6133_C2687793.pdf"
+		(property "Datasheet" "https://www.lcsc.com/datasheet/lcsc_datasheet_2409291808_Bardeen-Micro--BDR6133_C2687793.pdf"
 			(at 254 147.32 0)
 			(effects
@@
 			)
 		)
-		(property "Description" ""
+		(property "Description" "H-Bridge driver, 2.8A, 2V to 24V, PWM input, ESOP8"
 			(at 247.65 123.19 0)
 			(effects
