File: KiCad/v0.2/RP2040_minimal_Decoder.kicad_sch (KiCad schematic)
At the start: 64 parts, among them J1 T0, J10 2, J11 3, J12 4, J13 5, J14 +V, J15 M_OUT_B, J16 M_OUT_A, J17 GND, J18 SWCLK, J19 SWDIO, J2 Conn_01x02, J2 T1, J20 RUN, J3 0, J7 +3V3, J8 0, J9 1, Q1 T2N7002BK, Q2 T2N7002BK, Q3 T2N7002BK, Q4 T2N7002BK, Q5 T2N7002BK, U1 NCP1117-3.3_SOT223, U2 BDR6133, U2 W25Q128JVS, U3 RP2040, Y1 ABLS-12.000MHZ-B4-T

Commit message: cleaning up PCB
Parts:
- removed H4: MountingHole, MountingHole:MountingHole_2.7mm_M2.5, symbol Mechanical:MountingHole
- C1, C17, C4: footprint Capacitor_SMD:C_0805_2012Metric -> Capacitor_SMD:C_0805_2012Metric_Pad1.18x1.45mm_HandSolder
- C10, C11, C12, C13, C14, C15, C16, C2, C3, C5, C6, C7, C8, C9: footprint Capacitor_SMD:C_0402_1005Metric -> Capacitor_SMD:C_0805_2012Metric_Pad1.18x1.45mm_HandSolder
- J10, J11, J12, J13, J14, J15, J16, J17, J18, J19, J20, J3, J7, J8, J9: footprint TestPoint:TestPoint_Pad_D2.0mm -> TestPoint:TestPoint_Pad_D1.5mm
- R1, R2, R5, R6, R7, R8: footprint Resistor_SMD:R_0402_1005Metric -> Resistor_SMD:R_0805_2012Metric_Pad1.20x1.40mm_HandSolder
- U2: footprint Package_SO:SOIC-8-1EP_3.9x4.9mm_P1.27mm_EP2.41x3.3mm_ThermalVias -> User:SOIC-8-1EP_3.9x4.9mm_P1.27mm_EP2.41x3.3mm_BigThermalVias
- U3: footprint RP2040_minimal:RP2040-QFN-56 -> User:QFN-56-1EP_7x7mm_P0.4mm_EP3.2x3.2mm_BigThermalVias
- Y1: footprint RP2040_minimal:Crystal_SMD_HC49-US -> Crystal:Crystal_SMD_HC49-SD
Connections:
- net GPIO21: now also U3.37 (GPIO25); no longer U3.41 (GPIO29_ADC3)
- net GPIO22: now also U3.38 (GPIO26_ADC0); no longer U3.37 (GPIO25)
- net GPIO23: now also U3.39 (GPIO27_ADC1); no longer U3.38 (GPIO26_ADC0)
- net GPIO28_ADC2: now also U3.41 (GPIO29_ADC3); no longer U3.40 (GPIO28_ADC2)
- net GPIO29_ADC3: now also U3.40 (GPIO28_ADC2); no longer U3.39 (GPIO27_ADC1)
Other:
- note added: "I have intentionally not relabelled the GPIO nets as they may have been referenced elsewhere and would need to be re-mapped."
- company: Raspberry Pi (Trading) Ltd -> (none)
- title: RP2040 Minimal Design Example -> RP2040 Decoder
