File: KiCad/v0.1/RP2040-Decoder.kicad_pcb (KiCad board)
At the start: 2 copper layers, 85.1 x 97.8 mm, 56 parts, among them J1 T0, J10 2, J11 3, J12 4, J13 5, J14 +V, J15 M_OUT_B, J16 M_OUT_A, J17 GND, J18 SWCLK, J19 SWDIO, J2 T1, J20 RUN, J3 0, J4 1, J5 2, J6 3, J7 +3V3, J8 0, J9 1, Q1 T2N7002BK, Q2 T2N7002BK, Q3 T2N7002BK, Q4 T2N7002BK, Q5 T2N7002BK, U1 PJ75AL33SA, U2 BDR6133, U3 W25Q64JVSSIQ, U4 RP2040, Y1 X322512MSB4SI

Commit message: restore v0.1
Parts:
- added C9: 100n, RP2040-Decoder_Additional_Footprints:C_0603_1608Metric, F.Cu at (149.1, 105.3)
- C1, C14, C16, C17, C2: footprint Capacitor_SMD:C_0603_1608Metric -> RP2040-Decoder_Additional_Footprints:C_0603_1608Metric
- C10, C11, C12, C13, C15, C3, C4, C7, C8: footprint Capacitor_SMD:C_0402_1005Metric -> RP2040-Decoder_Additional_Footprints:C_0603_1608Metric
- C5, C6: value 1u -> 10u; footprint Capacitor_SMD:C_0402_1005Metric -> RP2040-Decoder_Additional_Footprints:C_0603_1608Metric
- J1, J10, J11, J12, J13, J14, J15, J16, J17, J18, J19, J2, J20, J3, J4, J5, J6, J7, J8, J9: moved to B.Cu
- moved J14 64.0 mm to (154.9, 99.0), turned to 180 degrees
- moved U2 62.9 mm to (159.8, 93.7), turned to -90 degrees
- moved J3 61.8 mm to (156.5, 108.3)
- moved J15 61.8 mm to (157.0, 92.0), turned to 180 degrees
- moved J6 60.6 mm to (156.6, 104.9)
- moved R9 59.7 mm to (139.0, 109.3), turned to 180 degrees
- moved J17 59.3 mm to (154.9, 101.6), turned to 180 degrees
- moved Q2 57.8 mm to (156.6, 108.3)
- moved C17 57.1 mm to (153.9, 108.4), turned to -90 degrees
- moved J4 57.0 mm to (160.5, 108.3)
- moved J5 56.9 mm to (160.5, 104.9)
- moved Q5 56.6 mm to (156.6, 104.9)
- moved J8 56.0 mm to (140.4, 98.9), turned to 180 degrees
- moved R1 55.9 mm to (150.1, 91.5), turned to -90 degrees
- moved R3 54.9 mm to (149.5, 97.6), turned to -90 degrees
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Routing:
- net +3V3: track 14.1 -> 92.6 mm, vias 0 -> 12
- net +V: track 0.00 -> 34.5 mm, vias 0 -> 9
- net Net-(D1-Pad1): track 0.00 -> 27.9 mm, vias 0 -> 9
- net Net-(R4-Pad1): track 0.00 -> 22.0 mm
- net Net-(R9-Pad2): track 0.00 -> 20.3 mm, vias 0 -> 2
- net /GPIO21: track 2.17 -> 20.5 mm, vias 0 -> 4
- net /ADC_EMF_A: track 0.00 -> 17.6 mm, vias 0 -> 2
- net /ADC_EMF_B: track 0.00 -> 16.9 mm, vias 0 -> 2
- net /GPIO22: track 3.97 -> 19.5 mm, vias 0 -> 2
- net Net-(U3-Pad7): track 0.00 -> 14.6 mm
- net Net-(U3-Pad5): track 0.00 -> 14.5 mm
- net /GPIO23: track 3.51 -> 17.9 mm, vias 0 -> 2
- net Net-(D1-Pad2): track 0.00 -> 13.1 mm, vias 0 -> 4
- net /GPIO25: track 2.84 -> 14.6 mm
- net /GPIO26: track 2.27 -> 13.8 mm
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- added copper zone on F.Cu, net GND
Other:
- board size 85.1 x 97.8 mm -> 25 x 20 mm
- board text added: "AUX"
- board text added: "DEBUG"
- board text added: "GPIO"
- board text added: "Gabriel Koppenstein RP2040-Decoder"
- board text added: "M"
- board text added: "Rev. 0.3"
