File: KiCad/v0.1/RP2040-Decoder.kicad_sch (KiCad schematic)
At the start: 56 parts, among them J1 T0, J10 2, J11 3, J12 4, J13 5, J14 +V, J15 M_OUT_B, J16 M_OUT_A, J17 GND, J18 SWCLK, J19 SWDIO, J2 T1, J20 RUN, J3 0, J4 1, J5 2, J6 3, J7 +3V3, J8 0, J9 1, Q1 T2N7002BK, Q2 T2N7002BK, Q3 T2N7002BK, Q4 T2N7002BK, Q5 T2N7002BK, U1 PJ75AL33SA, U2 BDR6133, U3 W25Q64JVSSIQ, U4 RP2040, Y1 X322512MSB4SI

Commit message: restore v0.1
Parts:
- added C9: 100n, RP2040-Decoder_Additional_Footprints:C_0603_1608Metric, symbol Device:C
- C1, C14, C16, C17, C2: footprint Capacitor_SMD:C_0603_1608Metric -> RP2040-Decoder_Additional_Footprints:C_0603_1608Metric
- C10, C11, C12, C13, C15, C3, C4, C7, C8: footprint Capacitor_SMD:C_0402_1005Metric -> RP2040-Decoder_Additional_Footprints:C_0603_1608Metric
- C5, C6: value 1u -> 10u; footprint Capacitor_SMD:C_0402_1005Metric -> RP2040-Decoder_Additional_Footprints:C_0603_1608Metric
Connections:
- net +3V3: now also C9.1
- net GND: now also C9.2
Changed lines of the file:
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@@
   (junction (at 20.32 153.67) (diameter 0) (color 0 0 0 0)
   )
+  (junction (at 133.35 67.31) (diameter 0) (color 0 0 0 0)
+  )
   (junction (at 102.87 67.31) (diameter 0) (color 0 0 0 0)
   )
@@
   )
   (junction (at 246.38 121.92) (diameter 0) (color 0 0 0 0)
+  )
+  (junction (at 133.35 77.47) (diameter 0) (color 0 0 0 0)
   )
   (junction (at 123.19 77.47) (diameter 0) (color 0 0 0 0)
@@
     (stroke (width 0) (type default))
   )
-  (wire (pts (xy 123.19 77.47) (xy 143.51 77.47))
+  (wire (pts (xy 133.35 77.47) (xy 123.19 77.47))
     (stroke (width 0) (type default))
   )
@@
     (stroke (width 0) (type default))
   )
+  (wire (pts (xy 143.51 77.47) (xy 133.35 77.47))
+    (stroke (width 0) (type default))
+  )
   (wire (pts (xy 76.2 30.48) (xy 72.39 30.48))
     (stroke (width 0) (type default))
@@
     (stroke (width 0) (type default))
   )
+  (wire (pts (xy 123.19 67.31) (xy 133.35 67.31))
+    (stroke (width 0) (type default))
+  )
   (wire (pts (xy 137.16 116.84) (xy 146.05 116.84))
     (stroke (width 0) (type default))
@@
     (stroke (width 0) (type default))
   )
+  (wire (pts (xy 133.35 67.31) (xy 133.35 68.58))
+    (stroke (width 0) (type default))
+  )
   (wire (pts (xy 83.82 38.1) (xy 83.82 48.26))
     (stroke (width 0) (type default))
@@
     (stroke (width 0) (type default))
   )
-  (wire (pts (xy 123.19 67.31) (xy 143.51 67.31))
+  (wire (pts (xy 133.35 67.31) (xy 143.51 67.31))
     (stroke (width 0) (type default))
   )
@@
   )
   (wire (pts (xy 137.16 114.3) (xy 146.05 114.3))
+    (stroke (width 0) (type default))
+  )
+  (wire (pts (xy 133.35 76.2) (xy 133.35 77.47))
     (stroke (width 0) (type default))
   )
@@
       (effects (font (size 1.27 1.27)) (justify left))
     )
-    (property "Value" "1u" (at 105.791 73.533 0)
-      (effects (font (size 1.27 1.27)) (justify left))
-    )
-    (property "Footprint" "Capacitor_SMD:C_0402_1005Metric" (at 103.8352 76.2 0)
+    (property "Value" "10u" (at 105.791 73.533 0)
+      (effects (font (size 1.27 1.27)) (justify left))
+    )
+    (property "Footprint" "RP2040-Decoder_Additional_Footprints:C_0603_1608Metric" (at 103.8352 76.2 0)
       (effects (font (size 1.27 1.27)) hide)
     )
@@
       (effects (font (size 1.27 1.27)) (justify left))
     )
-    (property "Value" "1u" (at 80.391 73.533 0)
-      (effects (font (size 1.27 1.27)) (justify left))
-    )
-    (property "Footprint" "Capacitor_SMD:C_0402_1005Metric" (at 78.4352 76.2 0)
+    (property "Value" "10u" (at 80.391 73.533 0)
+      (effects (font (size 1.27 1.27)) (justify left))
+    )
+    (property "Footprint" "RP2040-Decoder_Additional_Footprints:C_0603_1608Metric" (at 78.4352 76.2 0)
       (effects (font (size 1.27 1.27)) hide)
     )
@@
       (effects (font (size 1.27 1.27)) (justify left))
     )
-    (property "Footprint" "Capacitor_SMD:C_0402_1005Metric" (at 115.951 74.7014 0)
+    (property "Footprint" "RP2040-Decoder_Additional_Footprints:C_0603_1608Metric" (at 115.951 74.7014 0)
       (effects (font (size 1.27 1.27)) (justify left) hide)
     )
@@
       (effects (font (size 1.27 1.27)) (justify left))
     )
-    (property "Footprint" "Capacitor_SMD:C_0402_1005Metric" (at 126.111 74.7014 0)
+    (property "Footprint" "RP2040-Decoder_Additional_Footprints:C_0603_1608Metric" (at 126.111 74.7014 0)
       (effects (font (size 1.27 1.27)) (justify left) hide)
     )
@@
     )
   )
+  (symbol (lib_id "Device:C") (at 133.35 72.39 0) (unit 1)
+    (in_bom yes) (on_board yes) (dnp no)
+    (property "Reference" "C9" (at 136.271 71.2216 0)
+      (effects (font (size 1.27 1.27)) (justify left))
+    )
+    (property "Value" "100n" (at 136.271 73.533 0)
+      (effects (font (size 1.27 1.27)) (justify left))
+    )
+    (property "Footprint" "RP2040-Decoder_Additional_Footprints:C_0603_1608Metric" (at 136.271 74.7014 0)
+      (effects (font (size 1.27 1.27)) (justify left) hide)
+    )
+    (property "Datasheet" "~" (at 133.35 72.39 0)
+      (effects (font (size 1.27 1.27)) hide)
+    )
+    (pin "1")
+    (pin "2")
+    (instances
+      (project "RP2040-Decoder"
+        (path "/11d18738-0f49-4d63-b61c-22a93efd5959"
+          (reference "C9") (unit 1)
+        )
+      )
+    )
+  )
   (symbol (lib_id "Device:C") (at 143.51 72.39 0) (unit 1)
     (in_bom yes) (on_board yes) (dnp no)
@@
       (effects (font (size 1.27 1.27)) (justify left))
     )
-    (property "Footprint" "Capacitor_SMD:C_0402_1005Metric" (at 146.431 74.7014 0)
+    (property "Footprint" "RP2040-Decoder_Additional_Footprints:C_0603_1608Metric" (at 146.431 74.7014 0)
       (effects (font (size 1.27 1.27)) (justify left) hide)
     )
@@
       (effects (font (size 1.27 1.27)) (justify left))
     )
-    (property "Footprint" "Capacitor_SMD:C_0402_1005Metric" (at 70.231 74.7014 0)
+    (property "Footprint" "RP2040-Decoder_Additional_Footprints:C_0603_1608Metric" (at 70.231 74.7014 0)
       (effects (font (size 1.27 1.27)) (justify left) hide)
     )
@@
       (effects (font (size 1.27 1.27)) (justify left))
     )
-    (property "Footprint" "Capacitor_SMD:C_0402_1005Metric" (at 60.071 74.7014 0)
+    (property "Footprint" "RP2040-Decoder_Additional_Footprints:C_0603_1608Metric" (at 60.071 74.7014 0)
       (effects (font (size 1.27 1.27)) (justify left) hide)
     )
@@
       (effects (font (size 1.27 1.27)) (justify left))
     )
-    (property "Footprint" "Capacitor_SMD:C_0402_1005Metric" (at 156.591 74.7014 0)
+    (property "Footprint" "RP2040-Decoder_Additional_Footprints:C_0603_1608Metric" (at 156.591 74.7014 0)
       (effects (font (size 1.27 1.27)) (justify left) hide)
     )
@@
       (effects (font (size 1.27 1.27)) (justify left))
     )
-    (property "Footprint" "Capacitor_SMD:C_0402_1005Metric" (at 166.751 74.7014 0)
+    (property "Footprint" "RP2040-Decoder_Additional_Footprints:C_0603_1608Metric" (at 166.751 74.7014 0)
       (effects (font (size 1.27 1.27)) (justify left) hide)
     )
@@
       (effects (font (size 1.27 1.27)) (justify left))
     )
-    (property "Footprint" "Capacitor_SMD:C_0402_1005Metric" (at 176.911 74.7014 0)
+    (property "Footprint" "RP2040-Decoder_Additional_Footprints:C_0603_1608Metric" (at 176.911 74.7014 0)
       (effects (font (size 1.27 1.27)) (justify left) hide)
     )
@@
       (effects (font (size 1.27 1.27)) (justify left))
     )
-    (property "Footprint" "Capacitor_SMD:C_0603_1608Metric" (at 153.3652 95.25 0)
+    (property "Footprint" "RP2040-Decoder_Additional_Footprints:C_0603_1608Metric" (at 153.3652 95.25 0)
       (effects (font (size 1.27 1.27)) hide)
     )
@@
       (effects (font (size 1.27 1.27)) (justify left))
     )
-    (property "Footprint" "Capacitor_SMD:C_0402_1005Metric" (at 25.781 116.6114 0)
+    (property "Footprint" "RP2040-Decoder_Additional_Footprints:C_0603_1608Metric" (at 25.781 116.6114 0)
       (effects (font (size 1.27 1.27)) (justify left) hide)
     )
@@
       (effects (font (size 1.27 1.27)) (justify left))
     )
-    (property "Footprint" "Capacitor_SMD:C_0603_1608Metric" (at 23.241 162.3314 0)
+    (property "Footprint" "RP2040-Decoder_Additional_Footprints:C_0603_1608Metric" (at 23.241 162.3314 0)
       (effects (font (size 1.27 1.27)) (justify left) hide)
     )
@@
       (effects (font (size 1.27 1.27)) (justify left))
     )
-    (property "Footprint" "Capacitor_SMD:C_0603_1608Metric" (at 48.641 162.3314 0)
+    (property "Footprint" "RP2040-Decoder_Additional_Footprints:C_0603_1608Metric" (at 48.641 162.3314 0)
       (effects (font (size 1.27 1.27)) (justify left) hide)
     )
@@
       (effects (font (size 1.27 1.27)) (justify left))
     )
-    (property "Footprint" "Capacitor_SMD:C_0603_1608Metric" (at 71.4248 40.64 0)
+    (property "Footprint" "RP2040-Decoder_Additional_Footprints:C_0603_1608Metric" (at 71.4248 40.64 0)
       (effects (font (size 1.27 1.27)) hide)
     )
@@
       (effects (font (size 1.27 1.27)) (justify left))
     )
-    (property "Footprint" "Capacitor_SMD:C_0603_1608Metric" (at 49.8348 40.64 0)
+    (property "Footprint" "RP2040-Decoder_Additional_Footprints:C_0603_1608Metric" (at 49.8348 40.64 0)
       (effects (font (size 1.27 1.27)) hide)
     )
@@
     )
     (property "Value" "+3V3" (at 38.1 30.48 0)
-      (effects (font (size 1.27 1.27)) hide)
+      (effects (font (size 1.27 1.27)))
     )
     (property "Footprint" "TestPoint:TestPoint_Pad_D2.0mm" (at 44.45 30.48 0)
