File: KiCad/USB/RP2040-Decoder.kicad_sch (KiCad schematic)
At the start: 75 parts, among them J1 T0, J10 2, J11 3, J12 4, J13 5, J14 +V, J15 M_OUT_B, J16 M_OUT_A, J17 GND, J18 SWCLK, J19 SWDIO, J2 T1, J20 +3V3, J3 0, J4 1, J5 2, J6 3, J7 USB_C_Receptacle_USB2.0, J8 0, J9 1, Q1 T2N7002BK, Q2 T2N7002BK, Q3 T2N7002BK, Q4 T2N7002BK, Q5 T2N7002BK, SW1 TS-1088-AR02016, U2 LM4040C30FTA, U3 W25Q64JVSSIQ, U4 RP2040, U5 DRV8874PWPR, U6 AP7381-33Y-13, Y1 X322512MSB4SI

Commit message: Changes to schematic, Created PCB
Parts:
- added J21: SWDIO, TestPoint:TestPoint_Pad_D2.0mm, symbol Connector:Conn_01x01_Male
- added R17: 1k, RP2040-Decoder_Additional_Footprints:R_0603_1608Metric, symbol Device:R
- J7: footprint RP2040-Decoder_Additional_Footprints:USB_C_Receptacle_HRO_TYPE-C-31-M-12 -> Connector_USB:USB_C_Receptacle_HRO_TYPE-C-31-M-12; Datasheet original reference (none) -> https://datasheet.lcsc.com/lcsc/2205251630_Korean-Hroparts-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
Connections:
- net at R4.1, U3.1 (~{CS}), U4.56 (QSPI_SS): now also R17.1
- net at U4.26 (RUN): now also J21.1 (Pin_1); no longer SW1.2
- new net: R17.2, SW1.2
Other:
- note added: "Disable Flash boot (forces USB boot)"
- note added: "MCU"
- note added: "Voltage Reference"
- moved on the sheet: C10, C11, C12, C13, C15, C16, C17, C18, C19, C20, C21, C3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

Commit message: added pcb constraints, changed designators, updated footprints and 3d-models, created board outline
Parts:
- C1: renamed from C22; footprint RP2040-Decoder_Additional_Footprints:C_0603_1608Metric -> RP2040-Decoder_Additional_Footprints:C_0603_1608Metric_Removed_Silkscreen
- C10: renamed from C13; footprint RP2040-Decoder_Additional_Footprints:C_0603_1608Metric -> RP2040-Decoder_Additional_Footprints:C_0603_1608Metric_Removed_Silkscreen
- C11: renamed from C7; footprint RP2040-Decoder_Additional_Footprints:C_0603_1608Metric -> RP2040-Decoder_Additional_Footprints:C_0603_1608Metric_Removed_Silkscreen
- C12: renamed from C8; footprint RP2040-Decoder_Additional_Footprints:C_0603_1608Metric -> RP2040-Decoder_Additional_Footprints:C_0603_1608Metric_Removed_Silkscreen
- C13: renamed from C9; footprint RP2040-Decoder_Additional_Footprints:C_0603_1608Metric -> RP2040-Decoder_Additional_Footprints:C_0603_1608Metric_Removed_Silkscreen
- C14: renamed from C10; footprint RP2040-Decoder_Additional_Footprints:C_0603_1608Metric -> RP2040-Decoder_Additional_Footprints:C_0603_1608Metric_Removed_Silkscreen
- C15: renamed from C11; footprint RP2040-Decoder_Additional_Footprints:C_0603_1608Metric -> RP2040-Decoder_Additional_Footprints:C_0603_1608Metric_Removed_Silkscreen
- C16: renamed from C12; footprint RP2040-Decoder_Additional_Footprints:C_0603_1608Metric -> RP2040-Decoder_Additional_Footprints:C_0603_1608Metric_Removed_Silkscreen
- C17: renamed from C6; footprint RP2040-Decoder_Additional_Footprints:C_0603_1608Metric -> RP2040-Decoder_Additional_Footprints:C_0603_1608Metric_Removed_Silkscreen
- C18: renamed from C15; footprint RP2040-Decoder_Additional_Footprints:C_0603_1608Metric -> RP2040-Decoder_Additional_Footprints:C_0603_1608Metric_Removed_Silkscreen
- C19: renamed from C16; footprint RP2040-Decoder_Additional_Footprints:C_0603_1608Metric -> RP2040-Decoder_Additional_Footprints:C_0603_1608Metric_Removed_Silkscreen
- C2: renamed from C14; footprint RP2040-Decoder_Additional_Footprints:C_0603_1608Metric -> RP2040-Decoder_Additional_Footprints:C_0603_1608Metric_Removed_Silkscreen
- C20: renamed from C17; footprint RP2040-Decoder_Additional_Footprints:C_0603_1608Metric -> RP2040-Decoder_Additional_Footprints:C_0603_1608Metric_Removed_Silkscreen
- C3: renamed from C20; footprint RP2040-Decoder_Additional_Footprints:C_0603_1608Metric -> RP2040-Decoder_Additional_Footprints:C_0603_1608Metric_Removed_Silkscreen
- C4: renamed from C19; footprint RP2040-Decoder_Additional_Footprints:C_0603_1608Metric -> RP2040-Decoder_Additional_Footprints:C_0603_1608Metric_Removed_Silkscreen
- C5: renamed from C18; footprint RP2040-Decoder_Additional_Footprints:C_0603_1608Metric -> RP2040-Decoder_Additional_Footprints:C_0603_1608Metric_Removed_Silkscreen
- C6: renamed from C21; footprint RP2040-Decoder_Additional_Footprints:C_0603_1608Metric -> RP2040-Decoder_Additional_Footprints:C_0603_1608Metric_Removed_Silkscreen
- C7: renamed from C3; footprint RP2040-Decoder_Additional_Footprints:C_0603_1608Metric -> RP2040-Decoder_Additional_Footprints:C_0603_1608Metric_Removed_Silkscreen
- C8: renamed from C4; footprint RP2040-Decoder_Additional_Footprints:C_0603_1608Metric -> RP2040-Decoder_Additional_Footprints:C_0603_1608Metric_Removed_Silkscreen
- C9: renamed from C5; footprint RP2040-Decoder_Additional_Footprints:C_0603_1608Metric -> RP2040-Decoder_Additional_Footprints:C_0603_1608Metric_Removed_Silkscreen
- J1, J2: symbol Connector:Conn_01x01_Male -> Connector:Conn_01x01_Pin
- J10: renamed from J9; footprint TestPoint:TestPoint_Pad_D2.0mm -> TestPoint:TestPoint_Pad_D1.0mm; symbol Connector:Conn_01x01_Male -> Connector:Conn_01x01_Pin
- J11: renamed from J10; footprint TestPoint:TestPoint_Pad_D2.0mm -> TestPoint:TestPoint_Pad_D1.0mm; symbol Connector:Conn_01x01_Male -> Connector:Conn_01x01_Pin
- J12: renamed from J11; footprint TestPoint:TestPoint_Pad_D2.0mm -> TestPoint:TestPoint_Pad_D1.0mm; symbol Connector:Conn_01x01_Male -> Connector:Conn_01x01_Pin
- J13: renamed from J12; footprint TestPoint:TestPoint_Pad_D2.0mm -> TestPoint:TestPoint_Pad_D1.0mm; symbol Connector:Conn_01x01_Male -> Connector:Conn_01x01_Pin
- J14: renamed from J13; footprint TestPoint:TestPoint_Pad_D2.0mm -> TestPoint:TestPoint_Pad_D1.0mm; symbol Connector:Conn_01x01_Male -> Connector:Conn_01x01_Pin
- J15: renamed from J14; symbol Connector:Conn_01x01_Male -> Connector:Conn_01x01_Pin
- J16: renamed from J15; symbol Connector:Conn_01x01_Male -> Connector:Conn_01x01_Pin
- J17: renamed from J16; symbol Connector:Conn_01x01_Male -> Connector:Conn_01x01_Pin
- J18: renamed from J17; symbol Connector:Conn_01x01_Male -> Connector:Conn_01x01_Pin
- J19: renamed from J18; footprint TestPoint:TestPoint_Pad_D2.0mm -> TestPoint:TestPoint_Pad_D1.0mm; symbol Connector:Conn_01x01_Male -> Connector:Conn_01x01_Pin
- J20: renamed from J19; footprint TestPoint:TestPoint_Pad_D2.0mm -> TestPoint:TestPoint_Pad_D1.0mm; symbol Connector:Conn_01x01_Male -> Connector:Conn_01x01_Pin
- J21: footprint TestPoint:TestPoint_Pad_D2.0mm -> TestPoint:TestPoint_Pad_D1.0mm; symbol Connector:Conn_01x01_Male -> Connector:Conn_01x01_Pin
- J3, J4, J5, J6: footprint TestPoint:TestPoint_Pad_D2.0mm -> TestPoint:TestPoint_Pad_D1.5mm; symbol Connector:Conn_01x01_Male -> Connector:Conn_01x01_Pin
- J7: renamed from J20; symbol Connector:Conn_01x01_Male -> Connector:Conn_01x01_Pin
- J8: renamed from J7; footprint Connector_USB:USB_C_Receptacle_HRO_TYPE-C-31-M-12 -> RP2040-Decoder_Additional_Footprints:USB_C_Receptacle_HRO_TYPE-C-31-M-12
- J9: renamed from J8; footprint TestPoint:TestPoint_Pad_D2.0mm -> TestPoint:TestPoint_Pad_D1.0mm; symbol Connector:Conn_01x01_Male -> Connector:Conn_01x01_Pin
- R1, R14, R2: footprint RP2040-Decoder_Additional_Footprints:R_0603_1608Metric -> RP2040-Decoder_Additional_Footprints:R_0603_1608Metric_Removed_Silkscreen
- R10: renamed from R12; footprint RP2040-Decoder_Additional_Footprints:R_0603_1608Metric -> RP2040-Decoder_Additional_Footprints:R_0603_1608Metric_Removed_Silkscreen
- R11: renamed from R17; footprint RP2040-Decoder_Additional_Footprints:R_0603_1608Metric -> RP2040-Decoder_Additional_Footprints:R_0603_1608Metric_Removed_Silkscreen
- R12: renamed from R18; footprint RP2040-Decoder_Additional_Footprints:R_0603_1608Metric -> RP2040-Decoder_Additional_Footprints:R_0603_1608Metric_Removed_Silkscreen
- R13: renamed from R19; footprint RP2040-Decoder_Additional_Footprints:R_0603_1608Metric -> RP2040-Decoder_Additional_Footprints:R_0603_1608Metric_Removed_Silkscreen
- R15: renamed from R11; footprint RP2040-Decoder_Additional_Footprints:R_0603_1608Metric -> RP2040-Decoder_Additional_Footprints:R_0603_1608Metric_Removed_Silkscreen
- R16: renamed from R13; footprint RP2040-Decoder_Additional_Footprints:R_0603_1608Metric -> RP2040-Decoder_Additional_Footprints:R_0603_1608Metric_Removed_Silkscreen
- R17: renamed from R8; footprint RP2040-Decoder_Additional_Footprints:R_0603_1608Metric -> RP2040-Decoder_Additional_Footprints:R_0603_1608Metric_Removed_Silkscreen
- R18: renamed from R4; footprint RP2040-Decoder_Additional_Footprints:R_0603_1608Metric -> RP2040-Decoder_Additional_Footprints:R_0603_1608Metric_Removed_Silkscreen
- R19: renamed from R9; footprint RP2040-Decoder_Additional_Footprints:R_0603_1608Metric -> RP2040-Decoder_Additional_Footprints:R_0603_1608Metric_Removed_Silkscreen
- R3: renamed from R7; footprint RP2040-Decoder_Additional_Footprints:R_0603_1608Metric -> RP2040-Decoder_Additional_Footprints:R_0603_1608Metric_Removed_Silkscreen
- R4: renamed from R15; footprint RP2040-Decoder_Additional_Footprints:R_0603_1608Metric -> RP2040-Decoder_Additional_Footprints:R_0603_1608Metric_Removed_Silkscreen
- R5: renamed from R16; footprint RP2040-Decoder_Additional_Footprints:R_0603_1608Metric -> RP2040-Decoder_Additional_Footprints:R_0603_1608Metric_Removed_Silkscreen
- R6: renamed from R5; footprint RP2040-Decoder_Additional_Footprints:R_0603_1608Metric -> RP2040-Decoder_Additional_Footprints:R_0603_1608Metric_Removed_Silkscreen
- R7: renamed from R3; footprint RP2040-Decoder_Additional_Footprints:R_0603_1608Metric -> RP2040-Decoder_Additional_Footprints:R_0603_1608Metric_Removed_Silkscreen
- R8: renamed from R6; footprint RP2040-Decoder_Additional_Footprints:R_0603_1608Metric -> RP2040-Decoder_Additional_Footprints:R_0603_1608Metric_Removed_Silkscreen
- R9: renamed from R10; footprint RP2040-Decoder_Additional_Footprints:R_0603_1608Metric -> RP2040-Decoder_Additional_Footprints:R_0603_1608Metric_Removed_Silkscreen
- U3: renamed from U5; footprint Package_SO:HTSSOP-16-1EP_4.4x5mm_P0.65mm_EP3.4x5mm_Mask2.46x2.31mm_ThermalVias -> RP2040-Decoder_Additional_Footprints:HTSSOP-16-1EP_4.4x5mm_P0.65mm_EP3.4x5mm_Mask2.46x2.31mm_ThermalVias
- U5: renamed from U4; footprint RP2040-Decoder_Additional_Footprints:QFN-56-1EP_7x7mm_P0.4mm_EP3.2x3.2mm -> Package_DFN_QFN:QFN-56-1EP_7x7mm_P0.4mm_EP3.2x3.2mm
- renumbered D3 to D1, D1 to D2, D4 to D3, D2 to D4, U6 to U1, U3 to U4
Other:
- note removed: "C5/C6 should be close to pin 45/44"
- title: RP2040-Decoder -> RP2040-Decoder (USB)

Commit message: USB PCB routing, minor changes to schematic
Parts:
- removed C16: 100n, RP2040-Decoder_Additional_Footprints:C_0603_1608Metric_Removed_Silkscreen, symbol Device:C
- removed R6: 6k8, RP2040-Decoder_Additional_Footprints:R_0603_1608Metric_Removed_Silkscreen, symbol Device:R
- C1, C2: footprint RP2040-Decoder_Additional_Footprints:C_0603_1608Metric_Removed_Silkscreen -> Capacitor_SMD:C_0805_2012Metric
- J21: value SWDIO -> RUN
- R1, R2: footprint RP2040-Decoder_Additional_Footprints:R_0603_1608Metric_Removed_Silkscreen -> Resistor_SMD:R_0805_2012Metric
Connections:
- net GPIO6 is gone; now on net GPIO25: U3.3 (NSLEEP)
- net GPIO7 is gone; now on net GPIO20: U3.16 (PMODE)
- net ADC_EMF_A: now also U5.41 (GPIO29_ADC3); no longer U5.40 (GPIO28_ADC2)
- net ADC_EMF_B: now also U5.40 (GPIO28_ADC2); no longer U5.41 (GPIO29_ADC3)
- net GPIO12: now also Q2.1 (G), U5.15 (GPIO12); no longer U3.4 (NFAULT)
- net GPIO22: now also U3.1 (EN/IN1); no longer U3.2 (PH/IN2)
- net GPIO23: now also U3.2 (PH/IN2); no longer U3.1 (EN/IN1)
- net GPIO24: now also U3.4 (NFAULT)
- net at J11.1 (Pin_1): now also U5.13 (GPIO10); no longer U5.4 (GPIO2)
- net at J9.1 (Pin_1): now also U5.11 (GPIO8); no longer U5.2 (GPIO0)
- net at J12.1 (Pin_1): now also U5.14 (GPIO11); no longer U5.5 (GPIO3)
- net GPIO13: now reaches U5.16 (GPIO13)
- net GPIO13: now also Q3.1 (G)
- net GPIO14: now reaches U5.17 (GPIO14)
- net GPIO14: now also Q4.1 (G)
- net GPIO15: now reaches U5.18 (GPIO15)
- net GPIO15: now also Q5.1 (G)
- net at J10.1 (Pin_1): now also U5.12 (GPIO9); no longer U5.3 (GPIO1)
- net GPIO20: now reaches U5.31 (GPIO20)
- net USB_D_MCU-: now reaches R13.2, U5.46 (USB_DM)
- net USB_D_MCU+: now reaches R12.2, U5.47 (USB_DP)
- removed net GPIO10: Q4.1 (G), U5.13 (GPIO10)
- removed net GPIO11: Q5.1 (G), U5.14 (GPIO11)
- net GPIO26: no longer names the net of U5.38 (GPIO26_ADC0)
- removed net GPIO8: Q2.1 (G), U5.11 (GPIO8)
- removed net GPIO9: Q3.1 (G), U5.12 (GPIO9)
Other:
- note added: "GPIO24 is pulled up internally in RP2040"
- moved on the sheet: C17, R12, R13
