File: KiCad/USB/RP2040-Decoder.kicad_pcb (KiCad board)
At the start: 4 copper layers, 0 parts

Commit message: added pcb constraints, changed designators, updated footprints and 3d-models, created board outline
Parts:
- added C1: 10u, RP2040-Decoder_Additional_Footprints:C_0603_1608Metric_Removed_Silkscreen, F.Cu at (72.1, 33.5)
- added C10: 100n, RP2040-Decoder_Additional_Footprints:C_0603_1608Metric_Removed_Silkscreen, F.Cu at (76.1, 36.0)
- added C11: 100n, RP2040-Decoder_Additional_Footprints:C_0603_1608Metric_Removed_Silkscreen, F.Cu at (76.1, 38.5)
- added C12: 100n, RP2040-Decoder_Additional_Footprints:C_0603_1608Metric_Removed_Silkscreen, F.Cu at (76.1, 41.0)
- added C13: 100n, RP2040-Decoder_Additional_Footprints:C_0603_1608Metric_Removed_Silkscreen, F.Cu at (76.1, 43.5)
- added C14: 100n, RP2040-Decoder_Additional_Footprints:C_0603_1608Metric_Removed_Silkscreen, F.Cu at (76.1, 46.0)
- added C15: 100n, RP2040-Decoder_Additional_Footprints:C_0603_1608Metric_Removed_Silkscreen, F.Cu at (76.1, 48.5)
- added C16: 100n, RP2040-Decoder_Additional_Footprints:C_0603_1608Metric_Removed_Silkscreen, F.Cu at (76.1, 51.0)
- added C17: 10u, RP2040-Decoder_Additional_Footprints:C_0603_1608Metric_Removed_Silkscreen, F.Cu at (80.1, 33.5)
- added C18: 100n, RP2040-Decoder_Additional_Footprints:C_0603_1608Metric_Removed_Silkscreen, F.Cu at (80.1, 36.0)
- added C19: 33p, RP2040-Decoder_Additional_Footprints:C_0603_1608Metric_Removed_Silkscreen, F.Cu at (80.1, 38.5)
- added C2: 10u, RP2040-Decoder_Additional_Footprints:C_0603_1608Metric_Removed_Silkscreen, F.Cu at (72.1, 36.0)
- added C20: 33p, RP2040-Decoder_Additional_Footprints:C_0603_1608Metric_Removed_Silkscreen, F.Cu at (80.1, 41.0)
- added C3: 10u, RP2040-Decoder_Additional_Footprints:C_0603_1608Metric_Removed_Silkscreen, F.Cu at (72.1, 38.5)
- added C4: 100n, RP2040-Decoder_Additional_Footprints:C_0603_1608Metric_Removed_Silkscreen, F.Cu at (72.1, 41.0)
- added C5: 100n, RP2040-Decoder_Additional_Footprints:C_0603_1608Metric_Removed_Silkscreen, F.Cu at (72.1, 43.5)
- added C6: 22n, RP2040-Decoder_Additional_Footprints:C_0603_1608Metric_Removed_Silkscreen, F.Cu at (72.1, 46.0)
- added C7: 100n, RP2040-Decoder_Additional_Footprints:C_0603_1608Metric_Removed_Silkscreen, F.Cu at (72.1, 48.5)
- added C8: 100n, RP2040-Decoder_Additional_Footprints:C_0603_1608Metric_Removed_Silkscreen, F.Cu at (72.1, 51.0)
- added C9: 10u, RP2040-Decoder_Additional_Footprints:C_0603_1608Metric_Removed_Silkscreen, F.Cu at (76.1, 33.5)
- added D1: SS54, Diode_SMD:D_SMA, F.Cu at (66.1, 18.3)
- added D2: SS54, Diode_SMD:D_SMA, F.Cu at (66.1, 22.8)
- added D3: SS54, Diode_SMD:D_SMA, F.Cu at (66.1, 27.4)
- added D4: SS54, Diode_SMD:D_SMA, F.Cu at (66.1, 31.9)
- added D5: SS54, Diode_SMD:D_SMA, F.Cu at (66.1, 36.5)
- added J1: T0, TestPoint:TestPoint_Pad_D2.0mm, F.Cu at (72.1, 18.0)
- added J10: 1, TestPoint:TestPoint_Pad_D1.0mm, F.Cu at (80.2, 18.0)
- added J11: 2, TestPoint:TestPoint_Pad_D1.0mm, F.Cu at (80.2, 22.1)
- added J12: 3, TestPoint:TestPoint_Pad_D1.0mm, F.Cu at (80.2, 26.1)
- added J13: 4, TestPoint:TestPoint_Pad_D1.0mm, F.Cu at (80.2, 30.2)
- added J14: 5, TestPoint:TestPoint_Pad_D1.0mm, F.Cu at (84.3, 18.0)
- added J15: +V, TestPoint:TestPoint_Pad_D2.0mm, F.Cu at (84.3, 22.1)
- added J16: M_OUT_B, TestPoint:TestPoint_Pad_D2.0mm, F.Cu at (84.3, 26.1)
- added J17: M_OUT_A, TestPoint:TestPoint_Pad_D2.0mm, F.Cu at (84.3, 30.2)
- added J18: GND, TestPoint:TestPoint_Pad_D2.0mm, F.Cu at (88.3, 18.0)
- added J19: SWCLK, TestPoint:TestPoint_Pad_D1.0mm, F.Cu at (88.3, 22.1)
- added J2: T1, TestPoint:TestPoint_Pad_D2.0mm, F.Cu at (72.1, 22.1)
- added J20: SWDIO, TestPoint:TestPoint_Pad_D1.0mm, F.Cu at (88.3, 26.1)
- added J21: SWDIO, TestPoint:TestPoint_Pad_D1.0mm, F.Cu at (88.3, 30.2)
- added J3: 0, TestPoint:TestPoint_Pad_D1.5mm, F.Cu at (72.1, 26.1)
- added J4: 1, TestPoint:TestPoint_Pad_D1.5mm, F.Cu at (72.1, 30.2)
- added J5: 2, TestPoint:TestPoint_Pad_D1.5mm, F.Cu at (76.2, 18.0)
- added J6: 3, TestPoint:TestPoint_Pad_D1.5mm, F.Cu at (76.2, 22.1)
- added J7: +3V3, TestPoint:TestPoint_Pad_D2.0mm, F.Cu at (76.2, 26.1)
- added J8: USB_C_Receptacle_USB2.0, RP2040-Decoder_Additional_Footprints:USB_C_Receptacle_HRO_TYPE-C-31-M-12, F.Cu at (47.0, 30.0)
- added J9: 0, TestPoint:TestPoint_Pad_D1.0mm, F.Cu at (76.2, 30.2)
- added Q1: T2N7002BK, Package_TO_SOT_SMD:SOT-23, F.Cu at (59.6, 18.2)
- added Q2: T2N7002BK, Package_TO_SOT_SMD:SOT-23, F.Cu at (59.6, 22.7)
- added Q3: T2N7002BK, Package_TO_SOT_SMD:SOT-23, F.Cu at (59.6, 27.1)
- added Q4: T2N7002BK, Package_TO_SOT_SMD:SOT-23, F.Cu at (59.6, 31.6)
- added Q5: T2N7002BK, Package_TO_SOT_SMD:SOT-23, F.Cu at (59.6, 36.0)
- added R1: 6k8, RP2040-Decoder_Additional_Footprints:R_0603_1608Metric_Removed_Silkscreen, F.Cu at (80.1, 43.5)
- added R10: 6k8, RP2040-Decoder_Additional_Footprints:R_0603_1608Metric_Removed_Silkscreen, F.Cu at (84.1, 46.0)
- added R11: 1k, RP2040-Decoder_Additional_Footprints:R_0603_1608Metric_Removed_Silkscreen, F.Cu at (84.1, 48.5)
- added R12: 27R, RP2040-Decoder_Additional_Footprints:R_0603_1608Metric_Removed_Silkscreen, F.Cu at (84.1, 51.0)
- added R13: 27R, RP2040-Decoder_Additional_Footprints:R_0603_1608Metric_Removed_Silkscreen, F.Cu at (88.2, 33.5)
- added R14: 1k, RP2040-Decoder_Additional_Footprints:R_0603_1608Metric_Removed_Silkscreen, F.Cu at (88.2, 36.0)
- added R15: 1k, RP2040-Decoder_Additional_Footprints:R_0603_1608Metric_Removed_Silkscreen, F.Cu at (88.2, 38.5)
- added R16: 1k, RP2040-Decoder_Additional_Footprints:R_0603_1608Metric_Removed_Silkscreen, F.Cu at (88.2, 41.0)
- added R17: 1k, RP2040-Decoder_Additional_Footprints:R_0603_1608Metric_Removed_Silkscreen, F.Cu at (88.2, 43.5)
- added R18: DNF, RP2040-Decoder_Additional_Footprints:R_0603_1608Metric_Removed_Silkscreen, F.Cu at (88.2, 46.0)
- added R19: 1k, RP2040-Decoder_Additional_Footprints:R_0603_1608Metric_Removed_Silkscreen, F.Cu at (88.2, 48.5)
- added R2: 6k8, RP2040-Decoder_Additional_Footprints:R_0603_1608Metric_Removed_Silkscreen, F.Cu at (80.1, 46.0)
- added R3: 6k8, RP2040-Decoder_Additional_Footprints:R_0603_1608Metric_Removed_Silkscreen, F.Cu at (80.1, 48.5)
- added R4: 5k1, RP2040-Decoder_Additional_Footprints:R_0603_1608Metric_Removed_Silkscreen, F.Cu at (80.1, 51.0)
- added R5: 5k1, RP2040-Decoder_Additional_Footprints:R_0603_1608Metric_Removed_Silkscreen, F.Cu at (84.1, 33.5)
- added R6: 6k8, RP2040-Decoder_Additional_Footprints:R_0603_1608Metric_Removed_Silkscreen, F.Cu at (84.1, 36.0)
- added R7: 0R, RP2040-Decoder_Additional_Footprints:R_0603_1608Metric_Removed_Silkscreen, F.Cu at (84.1, 38.5)
- added R8: 1k2, RP2040-Decoder_Additional_Footprints:R_0603_1608Metric_Removed_Silkscreen, F.Cu at (84.1, 41.0)
- added R9: 6k8, RP2040-Decoder_Additional_Footprints:R_0603_1608Metric_Removed_Silkscreen, F.Cu at (84.1, 43.5)
- added SW1: TS-1088-AR02016, RP2040-Decoder_Additional_Footprints:TS-1088-AR02016 _footprint, F.Cu at (65.3, 40.9)
- added U1: AP7381-33Y-13, Package_TO_SOT_SMD:SOT-89-3, F.Cu at (65.4, 46.1)
- added U2: LM4040C30FTA, Package_TO_SOT_SMD:SOT-23, F.Cu at (59.6, 40.5)
- added U3: DRV8874PWPR, RP2040-Decoder_Additional_Footprints:HTSSOP-16-1EP_4.4x5mm_P0.65mm_EP3.4x5mm_Mask2.46x2.31mm_ThermalVias, F.Cu at (35.9, 23.3)
- added U4: W25Q64JVSSIQ, RP2040-Decoder_Additional_Footprints:SOIC-8_5.23x5.23mm_P1.27mm, F.Cu at (25.0, 23.0)
- added U5: RP2040, Package_DFN_QFN:QFN-56-1EP_7x7mm_P0.4mm_EP3.2x3.2mm, F.Cu at (26.8, 32.8)
- added Y1: X322512MSB4SI, Crystal:Crystal_SMD_3225-4Pin_3.2x2.5mm, F.Cu at (64.6, 51.4)
Other:
- board outline added: 30 x 20 mm

Commit message: USB PCB routing, minor changes to schematic
Parts:
- removed C16: 100n, RP2040-Decoder_Additional_Footprints:C_0603_1608Metric_Removed_Silkscreen
- removed R6: 6k8, RP2040-Decoder_Additional_Footprints:R_0603_1608Metric_Removed_Silkscreen
- C1, C2: footprint RP2040-Decoder_Additional_Footprints:C_0603_1608Metric_Removed_Silkscreen -> Capacitor_SMD:C_0805_2012Metric; moved to B.Cu
- D1, D2, D3, D4, D5, J1, J15, J16, J17, J18, J2, J3, J4, J5, J6, J7, Q1, Q2, Q3, Q4, Q5, U1: moved to B.Cu
- J21: value SWDIO -> RUN
- R1, R2: footprint RP2040-Decoder_Additional_Footprints:R_0603_1608Metric_Removed_Silkscreen -> Resistor_SMD:R_0805_2012Metric; moved to B.Cu
- moved J19 67.9 mm to (20.7, 27.8)
- moved J20 67.7 mm to (20.7, 29.9)
- moved J21 67.7 mm to (20.7, 31.9)
- moved R17 66.6 mm to (22.1, 34.7)
- moved R16 66.2 mm to (22.1, 36.4)
- moved R19 64.7 mm to (26.0, 30.4), turned to -90 degrees
- moved R10 62.5 mm to (22.1, 38.1)
- moved C20 59.1 mm to (23.3, 24.7)
- moved J5 57.5 mm to (20.8, 33.5), turned to 180 degrees
- moved C19 57.3 mm to (23.3, 30.9), turned to 180 degrees
- moved R18 55.5 mm to (38.8, 20.7)
- moved R2 55.2 mm to (25.5, 37.8), turned to 90 degrees
- moved R11 55.0 mm to (36.3, 21.4), turned to 90 degrees
- moved J6 54.1 mm to (23.3, 33.5), turned to 180 degrees
- moved J17 53.9 mm to (30.5, 33.0), turned to 90 degrees
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Connections:
- net Net-(U5-USB_DM) renamed /USB_D_MCU-
- net Net-(U5-USB_DP) renamed /USB_D_MCU+
- Q2 pad 1: /GPIO8 -> /GPIO12
- Q3 pad 1: /GPIO9 -> /GPIO13
- Q4 pad 1: /GPIO10 -> /GPIO14
- Q5 pad 1: /GPIO11 -> /GPIO15
- U3 pad 1: /GPIO23 -> /GPIO22
- U3 pad 16: /GPIO7 -> /GPIO20
- U3 pad 2: /GPIO22 -> /GPIO23
- U3 pad 3: /GPIO6 -> /GPIO25
- U3 pad 4: /GPIO12 -> /GPIO24
- U5 pad 11: /GPIO8 -> Net-(J9-Pin_1)
- U5 pad 12: /GPIO9 -> Net-(J10-Pin_1)
- U5 pad 13: /GPIO10 -> Net-(J11-Pin_1)
- U5 pad 14: /GPIO11 -> Net-(J12-Pin_1)
- U5 pad 15: unconnected-(U5-GPIO12-Pad15) -> /GPIO12
- U5 pad 16: unconnected-(U5-GPIO13-Pad16) -> /GPIO13
- U5 pad 17: unconnected-(U5-GPIO14-Pad17) -> /GPIO14
- U5 pad 18: unconnected-(U5-GPIO15-Pad18) -> /GPIO15
- U5 pad 2: Net-(J9-Pin_1) -> unconnected-(U5-GPIO0-Pad2)
- U5 pad 3: Net-(J10-Pin_1) -> unconnected-(U5-GPIO1-Pad3)
- U5 pad 31: unconnected-(U5-GPIO20-Pad31) -> /GPIO20
- U5 pad 38: /GPIO26 -> unconnected-(U5-GPIO26_ADC0-Pad38)
- U5 pad 4: Net-(J11-Pin_1) -> unconnected-(U5-GPIO2-Pad4)
- U5 pad 40: /ADC_EMF_A -> /ADC_EMF_B
- U5 pad 41: /ADC_EMF_B -> /ADC_EMF_A
- U5 pad 5: Net-(J12-Pin_1) -> unconnected-(U5-GPIO3-Pad5)
Routing:
- net +3V3: track 0.00 -> 28.2 mm, vias 0 -> 4
- net /VREF: track 0.00 -> 26.2 mm, vias 0 -> 2
- net +V: track 0.00 -> 24.1 mm
- net Net-(D1-K): track 0.00 -> 22.2 mm
- net Net-(U4-DO(IO1)): track 0.00 -> 18.7 mm, vias 0 -> 2
- net Net-(U4-~{CS}): track 0.00 -> 18.0 mm, vias 0 -> 2
- net Net-(U4-IO2): track 0.00 -> 17.2 mm
- net Net-(R11-Pad2): track 0.00 -> 16.8 mm, vias 0 -> 2
- net /ADC_EMF_B: track 0.00 -> 15.8 mm, vias 0 -> 2
- net +1V1: track 0.00 -> 15.7 mm, vias 0 -> 2
- net Net-(J19-Pin_1): track 0.00 -> 13.4 mm
- net /GPIO20: track 0.00 -> 13.1 mm
- net /GPIO25: track 0.00 -> 13.0 mm
- net /MOTOR_OUT_A: track 0.00 -> 13.0 mm, vias 0 -> 4
- net /GPIO23: track 0.00 -> 12.9 mm, vias 0 -> 2
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
Commit message: PCB Routing
Routing:
- net GND: track 3.46 -> 26.4 mm, vias 3 -> 21
- net +3V3: track 28.2 -> 35.3 mm, vias 4 -> 9
- net +V: track 24.1 -> 31.3 mm, vias 0 -> 1
- net +1V1: track 15.7 -> 21.0 mm, vias 2 -> 0
- net /MOTOR_OUT_B: track 10.7 -> 13.8 mm
- net Net-(U5-XIN): track 8.84 -> 7.63 mm
- net /GPIO23: track 12.9 -> 11.8 mm
- net /GPIO20: track 13.1 -> 14.0 mm
- net Net-(D3-K): track 7.46 -> 8.29 mm
- net Net-(D1-K): track 22.2 -> 22.9 mm
- net /GPIO24: track 12.8 -> 12.1 mm
- net Net-(U4-~{CS}): track 18.0 -> 18.7 mm
- added copper zone on In2.Cu, net +3V3
- added copper zone on In1.Cu, net GND

Commit message: PCB routing
Parts:
- moved C12 14.1 mm to (40.3, 43.0)
- moved C3 14.1 mm to (35.2, 45.1)
- moved C4 14.1 mm to (36.7, 45.1)
- moved D4 14.1 mm to (50.9, 37.7)
- moved J12 14.1 mm to (36.9, 32.2)
- moved J15 14.1 mm to (47.6, 41.2)
- moved J2 14.1 mm to (47.6, 35.2)
- moved J8 14.1 mm to (57.0, 41.2)
- moved Q2 14.1 mm to (32.0, 35.7)
- moved Q3 14.1 mm to (36.5, 35.7)
- moved C1 14.1 mm to (44.9, 39.6)
- moved C10 14.1 mm to (48.8, 36.6)
- moved C11 14.1 mm to (43.8, 43.0)
- moved C13 14.1 mm to (36.0, 34.4)
- moved C14 14.1 mm to (41.0, 31.4)
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Routing:
- net +3V3: track 35.3 -> 43.9 mm, vias 9 -> 13
- net GND: track 26.4 -> 26.1 mm, vias 21 -> 20
