File: KiCad/USB/RP2040-Decoder.kicad_pcb (KiCad board)
At the start: 4 copper layers, 25 x 20 mm, 68 parts, among them J1 Conn_01x01, J10 Conn_01x01, J11 Conn_01x01, J12 Conn_01x01, J13 Conn_01x01, J14 Conn_01x01, J15 Conn_01x01, J16 Conn_01x01, J17 Conn_01x01, J18 Conn_01x01, J19 Conn_01x01, J2 Conn_01x01, J20 Conn_01x01, J21 Conn_01x01, J3 USB_C_Receptacle_USB2.0_16P, J4 Conn_01x01, J5 Conn_01x01, J6 Conn_01x01, J7 Conn_01x01, J8 Conn_01x01, J9 Conn_01x01, Q1 Si1308EDL, Q2 Si1308EDL, Q3 Si1308EDL, Q4 Si1308EDL, Q5 Si1308EDL, SW1 YTS1T0162AWJ00, U1 MIC5200-3.3YS, U2 W25Q64JVSSIQ, U3 RP2040, U4 BDR6133, Y1 X322512MSB4SI

Commit message: Update README and add Revision attribute to PCB which updates Rev x.x silkscreen on the back side;
Other:
- board text added: "Rev. ${REVISION}"
- board text removed: "Rev. 1.0"
Changed lines of the file:
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@@
 	)
 	(paper "A4")
+	(title_block
+		(rev "1.1")
+	)
 	(layers
 		(0 "F.Cu" signal)
@@
 		)
 	)
-	(gr_text "Rev. 1.0"
+	(gr_text "Rev. ${REVISION}"
 		(at 150.3 107.7 0)
 		(layer "B.SilkS")
