File: KiCad/Rev_1_0/RP2040-Decoder.kicad_pcb (KiCad board)
At the start: 4 copper layers, 25 x 20 mm, 68 parts, among them J1 Conn_01x01, J10 Conn_01x01, J11 Conn_01x01, J12 Conn_01x01, J13 Conn_01x01, J14 Conn_01x01, J15 Conn_01x01, J16 Conn_01x01, J17 Conn_01x01, J18 Conn_01x01, J19 Conn_01x01, J2 Conn_01x01, J20 Conn_01x01, J21 Conn_01x01, J3 USB_C_Receptacle_USB2.0_16P, J4 Conn_01x01, J5 Conn_01x01, J6 Conn_01x01, J7 Conn_01x01, J8 Conn_01x01, J9 Conn_01x01, Q1 Si1308EDL, Q2 Si1308EDL, Q3 Si1308EDL, Q4 Si1308EDL, Q5 Si1308EDL, U1 MIC5200-3.3YS, U2 W25Q64JVSSIQ, U3 RP2040, U4 BDR6133, Y1 X322512MSB4SI

Commit message: Change C18 to be 0603 - 25V and rotate on PCB for easier soldering; Small logging changes; Speed step enums are actually used now for better clarity; Introduced cv_setup_check_done and flash_safe_execute_core_init_done flags for coordinating the two cores better; Incremented version no. CV_7 to 2;
Parts:
- C18: footprint Capacitor_SMD:C_0402_1005Metric -> Capacitor_SMD:C_0603_1608Metric
- moved C18 2.14 mm to (160.7, 92.7), turned to -90 degrees
- moved C17 0.30 mm to (158.9, 92.7)
Routing:
- net GND: track 4.35 -> 2.73 mm
Changed lines of the file:
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@@
 		(tags "SOIC SO")
 		(property "Reference" "U4"
-			(at -0.2 -4.3 -90)
-			(layer "F.SilkS")
+			(at 1.7 0 0)
+			(layer "B.SilkS")
 			(effects
 				(font
@@
 					(thickness 0.15)
 				)
+				(justify mirror)
 			)
 		)
 		(property "Value" "BDR6133"
-			(at 0 3.4 -90)
+			(at 0 3.4 90)
 			(layer "F.Fab")
 			(effects
@@
 		)
 		(property "Footprint" "RP2040-Decoder_Additional_Footprints:SOIC-8-1EP_3.9x4.9mm_P1.27mm_EP2.41x3.3mm_ThermalVias"
-			(at 0 0 -90)
+			(at 0 0 90)
 			(layer "F.Fab")
 			(hide yes)
@@
 		)
 		(property "Datasheet" "https://www.lcsc.com/datasheet/lcsc_datasheet_2409291808_Bardeen-Micro--BDR6133_C2687793.pdf"
-			(at 0 0 -90)
+			(at 0 0 90)
 			(layer "F.Fab")
 			(hide yes)
@@
 		)
 		(property "Description" "H-Bridge driver, 2.8A, 2V to 24V, PWM input, ESOP8"
-			(at 0 0 -90)
+			(at 0 0 90)
 			(layer "F.Fab")
 			(hide yes)
@@
 		(sheetname "Root")
 		(sheetfile "RP2040-Decoder.kicad_sch")
-		(attr smd)
 		(fp_line
 			(start -1.55 2.56)
@@
 		)
 		(fp_text user "${REFERENCE}"
-			(at 0 0 -90)
+			(at 0 0 90)
 			(layer "F.Fab")
 			(effects
@@
 		)
 	)
-	(footprint "Capacitor_SMD:C_0402_1005Metric"
+	(footprint "Capacitor_SMD:C_0603_1608Metric"
 		(layer "B.Cu")
-		(at 161.1 90.6)
-		(descr "Capacitor SMD 0402 (1005 Metric), square (rectangular) end terminal, IPC_7351 nominal, (Body size source: IPC-SM-782 page 76, https://www.pcb-3d.com/wordpress/wp-content/uploads/ipc-sm-782a_amendment_1_and_2.pdf), generated with kicad-footprint-generator")
+		(at 160.7 92.7 -90)
+		(descr "Capacitor SMD 0603 (1608 Metric), square (rectangular) end terminal, IPC_7351 nominal, (Body size source: IPC-SM-782 page 76, https://www.pcb-3d.com/wordpress/wp-content/uploads/ipc-sm-782a_amendment_1_and_2.pdf), generated with kicad-footprint-generator")
 		(tags "capacitor")
 		(property "Reference" "C18"
-			(at 0.8 3.3 -90)
+			(at -1 -1.2 -90)
 			(layer "B.SilkS")
 			(effects
@@
 		)
 		(property "Value" "10u"
-			(at 0 -1.16 0)
+			(at 0 -1.43 90)
 			(layer "B.Fab")
-			(hide yes)
 			(effects
 				(font
@@
 			)
 		)
-		(property "Footprint" "Capacitor_SMD:C_0402_1005Metric"
-			(at 0 0 180)
+		(property "Footprint" "Capacitor_SMD:C_0603_1608Metric"
+			(at 0 0 90)
 			(unlocked yes)
 			(layer "B.Fab")
@@
 		)
 		(property "Datasheet" ""
-			(at 0 0 180)
+			(at 0 0 90)
 			(unlocked yes)
 			(layer "B.Fab")
@@
 		)
 		(property "Description" ""
-			(at 0 0 180)
+			(at 0 0 90)
 			(unlocked yes)
 			(layer "B.Fab")
@@
 			)
 		)
-		(property "Voltage" "6V3"
-			(at 0 0 180)
+		(property "Voltage" "25V"
+			(at 0 0 -90)
 			(unlocked yes)
 			(layer "B.Fab")
@@
 		)
 		(property "Alternative Part" ""
-			(at 0 0 180)
+			(at 0 0 -90)
 			(unlocked yes)
 			(layer "B.Fab")
@@
 			)
 		)
-		(property "LCSC Part #" "C15525"
-			(at 0 0 0)
+		(property "LCSC Part #" "C96446"
+			(at 0 0 -90)
 			(unlocked yes)
 			(layer "B.Fab")
@@
 		)
 		(property "JLCPCB Rotation Offset" ""
-			(at 0 0 0)
+			(at 0 0 -90)
 			(unlocked yes)
 			(layer "B.Fab")
@@
 		(attr smd)
 		(fp_line
-			(start 0.107836 -0.36)
-			(end -0.107836 -0.36)
+			(start 0.14058 0.51)
+			(end -0.14058 0.51)
 			(stroke
 				(width 0.12)
@@
 		)
 		(fp_line
-			(start 0.107836 0.36)
-			(end -0.107836 0.36)
+			(start 0.14058 -0.51)
+			(end -0.14058 -0.51)
 			(stroke
 				(width 0.12)
@@
 		)
 		(fp_line
-			(start -0.91 -0.46)
-			(end 0.91 -0.46)
+			(start -1.48 0.73)
+			(end -1.48 -0.73)
 			(stroke
 				(width 0.05)
@@
 		)
 		(fp_line
-			(start -0.91 0.46)
-			(end -0.91 -0.46)
+			(start 1.48 0.73)
+			(end -1.48 0.73)
 			(stroke
 				(width 0.05)
@@
 		)
 		(fp_line
-			(start 0.91 -0.46)
-			(end 0.91 0.46)
+			(start -1.48 -0.73)
+			(end 1.48 -0.73)
 			(stroke
 				(width 0.05)
@@
 		)
 		(fp_line
-			(start 0.91 0.46)
-			(end -0.91 0.46)
+			(start 1.48 -0.73)
+			(end 1.48 0.73)
 			(stroke
 				(width 0.05)
@@
 		)
 		(fp_line
-			(start -0.5 -0.25)
-			(end 0.5 -0.25)
+			(start -0.8 0.4)
+			(end -0.8 -0.4)
 			(stroke
 				(width 0.1)
@@
 		)
 		(fp_line
-			(start -0.5 0.25)
-			(end -0.5 -0.25)
+			(start 0.8 0.4)
+			(end -0.8 0.4)
 			(stroke
 				(width 0.1)
@@
 		)
 		(fp_line
-			(start 0.5 -0.25)
-			(end 0.5 0.25)
+			(start -0.8 -0.4)
+			(end 0.8 -0.4)
 			(stroke
 				(width 0.1)
@@
 		)
 		(fp_line
-			(start 0.5 0.25)
-			(end -0.5 0.25)
+			(start 0.8 -0.4)
+			(end 0.8 0.4)
 			(stroke
 				(width 0.1)
@@
 		)
 		(fp_text user "${REFERENCE}"
-			(at 0 0 0)
+			(at 0 0 90)
 			(layer "B.Fab")
 			(effects
 				(font
-					(size 0.25 0.25)
-					(thickness 0.04)
+					(size 0.4 0.4)
+					(thickness 0.06)
 				)
 				(justify mirror)
@@
 		)
 		(pad "1" smd roundrect
-			(at -0.48 0)
-			(size 0.56 0.62)
+			(at -0.775 0 270)
+			(size 0.9 0.95)
 			(layers "B.Cu" "B.Paste" "B.Mask")
 			(roundrect_rratio 0.25)
@@
 		)
 		(pad "2" smd roundrect
-			(at 0.48 0)
-			(size 0.56 0.62)
+			(at 0.775 0 270)
+			(size 0.9 0.95)
 			(layers "B.Cu" "B.Paste" "B.Mask")
 			(roundrect_rratio 0.25)
@@
 			(pintype "passive")
 		)
-		(model "${KICAD8_3DMODEL_DIR}/Capacitor_SMD.3dshapes/C_0402_1005Metric.wrl"
+		(model "${KICAD8_3DMODEL_DIR}/Capacitor_SMD.3dshapes/C_0603_1608Metric.wrl"
 			(offset
 				(xyz 0 0 0)
@@
 	(footprint "Capacitor_SMD:C_0603_1608Metric"
 		(layer "B.Cu")
-		(at 159.2 92.7 -90)
+		(at 158.9 92.7 -90)
 		(descr "Capacitor SMD 0603 (1608 Metric), square (rectangular) end terminal, IPC_7351 nominal, (Body size source: IPC-SM-782 page 76, https://www.pcb-3d.com/wordpress/wp-content/uploads/ipc-sm-782a_amendment_1_and_2.pdf), generated with kicad-footprint-generator")
 		(tags "capacitor")
 		(property "Reference" "C17"
-			(at 2.9 0 0)
+			(at -0.9 1.1 90)
 			(layer "B.SilkS")
 			(effects
@@
 		(layer "B.Mask")
 	)
-	(gr_line
-		(start 161.7 92.1)
-		(end 161.7 90.5)
-		(stroke
-			(width 0.6)
-			(type default)
-		)
-		(layer "B.Mask")
-	)
 	(gr_poly
 		(pts
@@
 		(layer "B.Mask")
 	)
-	(gr_line
-		(start 161.7 90.7)
-		(end 161.7 92.1)
-		(stroke
-			(width 0.6)
-			(type default)
-		)
-		(layer "B.Mask")
-	)
 	(gr_rect
 		(start 137.5 90)
@@
 	)
 	(via
-		(at 160.425 92.1)
-		(size 0.4)
-		(drill 0.3)
-		(layers "F.Cu" "B.Cu")
-		(net 1)
-	)
-	(via
 		(at 144 99.3)
 		(size 0.4)
@@
 	)
 	(via
+		(at 160.425 90.5)
+		(size 0.4)
+		(drill 0.3)
+		(layers "F.Cu" "B.Cu")
+		(net 1)
+	)
+	(via
 		(at 153.686814 99.386814)
 		(size 0.4)
@@
 	)
 	(segment
+		(start 160.425 90.5)
+		(end 160.425 91.15)
+		(width 0.6)
+		(layer "B.Cu")
+		(net 1)
+	)
+	(segment
 		(start 139.025 101.575)
 		(end 139 101.6)
@@
 	)
 	(segment
-		(start 160.425 92.1)
-		(end 160.425 90.695)
+		(start 160.425 91.85)
+		(end 160.5 91.925)
 		(width 0.6)
 		(layer "B.Cu")
@@
 	)
 	(segment
+		(start 160.425 91.15)
+		(end 160.425 91.85)
+		(width 0.6)
+		(layer "B.Cu")
+		(net 1)
+	)
+	(segment
 		(start 141.4 98.225)
 		(end 139.625 98.225)
@@
 	)
 	(segment
-		(start 160.52 90.6)
-		(end 160.425 90.695)
-		(width 0.6)
-		(layer "B.Cu")
-		(net 1)
-	)
-	(segment
 		(start 141.4 98.225)
 		(end 145.725 98.225)
@@
 	)
 	(segment
-		(start 160.62 90.6)
-		(end 160.52 90.6)
-		(width 0.6)
-		(layer "B.Cu")
-		(net 1)
-	)
-	(segment
 		(start 145.725 98.225)
 		(end 146.2 98.7)
@@
 	)
 	(segment
-		(start 158.700306 91.925)
-		(end 158.228338 92.396968)
-		(width 0.6)
-		(layer "B.Cu")
-		(net 2)
-	)
-	(segment
 		(start 157.12 97.2)
 		(end 152.85 97.2)
@@
 	)
 	(segment
-		(start 159.175 91.9)
-		(end 159.2 91.925)
-		(width 0.6)
-		(layer "B.Cu")
-		(net 2)
-	)
-	(segment
 		(start 158.103032 92.396968)
-		(end 157.8 92.7)
+		(end 158.428032 92.396968)
 		(width 0.6)
 		(layer "B.Cu")
@@
 	)
 	(segment
-		(start 158.228338 92.396968)
-		(end 158.103032 92.396968)
+		(start 140.325 109.5)
+		(end 139.025 108.2)
 		(width 0.6)
 		(layer "B.Cu")
@@
 	)
 	(segment
-		(start 140.325 109.5)
-		(end 139.025 108.2)
+		(start 158.428032 92.396968)
+		(end 158.9 91.925)
 		(width 0.6)
 		(layer "B.Cu")
@@
 	)
 	(segment
-		(start 159.2 91.925)
-		(end 158.700306 91.925)
+		(start 152.85 97.2)
+		(end 156.1 97.2)
 		(width 0.6)
 		(layer "B.Cu")
@@
 	)
 	(segment
-		(start 152.85 97.2)
-		(end 156.1 97.2)
+		(start 157.852298 95.152298)
+		(end 157.852298 96.747702)
 		(width 0.6)
 		(layer "B.Cu")
@@
 	)
 	(segment
-		(start 157.852298 95.152298)
-		(end 157.852298 96.747702)
+		(start 157.8 92.7)
+		(end 158.103032 92.396968)
 		(width 0.6)
 		(layer "B.Cu")
@@
 	)
 	(segment
-		(start 161.58 90.6)
-		(end 161.7 90.6)
-		(width 0.6)
-		(layer "B.Cu")
-		(net 4)
-	)
-	(segment
 		(start 145.3 103.9)
 		(end 144.975 103.9)
@@
 		(layer "B.Cu")
 		(net 4)
-	)
-	(segment
-		(start 161.7 90.6)
-		(end 161.7 92.1)
-		(width 0.6)
-		(layer "B.Cu")
-		(net 4)

Commit message: Replaced solder bridge with tactile button; Fixed Footprint Rotation in position file; Fixed .gitignore for production outputs
Parts:
- removed JP1: SolderJumper_2_Open, Jumper:SolderJumper-2_P1.3mm_Open_RoundedPad1.0x1.5mm
- added SW1: YTS1T0162AWJ00, RP2040-Decoder_Additional_Footprints:SW_Push_1P1T_NO_Vertical_Wuerth_434133025816, B.Cu at (142.7, 95.5)
- turned R4 to 90 degrees
Connections:
- R4 pad 1: Net-(JP1-B) -> Net-(U2-~{CS})
- R4 pad 2: Net-(U2-~{CS}) -> Net-(R4-Pad2)
Routing:
- net Net-(R4-Pad2): track 0.00 -> 5.77 mm, vias 0 -> 1
- net Net-(JP1-B): track 2.11 -> 0.00 mm, vias 1 -> 0
